File: schematic/ALL.kicad_pcb (KiCad board)
At the start: 4 copper layers, 200.5 x 70.9 mm, 138 parts, among them CON1 USB-MICRO-B, IC1 ADM233L, IC2.1 L6208N, IC2.2 L6208N, IC2.3 L6208N, IC2.4 L6208N, IC2.5 L6208N, J1 DB9, J2 DB9, K1 CONN_3, P1 CONN_2, P10 TRD, P11 CONN_7, P12 CONN_12, P13 CONN_5, P14 CONN_2, P15 CONN_4, P16 CONN_7, P17 CONN_2, P18 CONN_2, P19 CONN_2, P2 CONN_4, P3 CONN_4, P4 CONN_4, P5 CONN_4, P6 CONN_4, P7 CONN_2, P8 CONN_2, P9 CONN_2, Q1 DTA114Y, Q2 8MHz, Q3 RO-1224, SW1 RESET, SW2 BOOT, U1 IPS5451, U2 TLE5205, U3 STM32F103, U4 USBLC6-2, U5 LM1117MPX-3.3

Commit message: PCB
Parts:
- R11, R22, R23, R24: moved to B.Cu
- R25: value 1.2k (II) -> 300 (II)
- moved R20 123.4 mm to (115.2, 93.3)
- moved P18 105.0 mm to (125.9, 79.8), turned to 270 degrees
- moved R19 94.1 mm to (110.1, 84.8), turned to 180 degrees
- moved U1 89.5 mm to (116.1, 86.6)
- moved R37 86.6 mm to (178.2, 130.3), turned to 270 degrees
- moved R39 80.1 mm to (110.1, 82.9)
- moved R38 67.6 mm to (158.6, 130.0), turned to 270 degrees
- moved P14 64.5 mm to (187.3, 142.2)
- moved R23 59.2 mm to (124.6, 110.6)
- moved U2 58.5 mm to (188.5, 130.5), turned to 270 degrees
- moved R24 54.4 mm to (129.2, 118.7)
- moved R22 53.1 mm to (129.2, 116.1)
- moved P8 34.7 mm to (170.1, 142.4)
- moved C4 32.2 mm to (217.7, 128.4), turned to 270 degrees
- moved R25 32.0 mm to (215.4, 141.5)
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Connections:
- C12 pad 2: +3.3V -> +5V
- Q1 pad 2: +3.3V -> +5V
- R13 pad 2: +5V -> +3.3V
- R14 pad 2: +5V -> +3.3V
- R15 pad 2: +5V -> +3.3V
- R16 pad 2: +5V -> +3.3V
- R20 pad 1: /STM32F103 module/DG_FEEDBACK -> /STM32F103 module/POW3_FEEDBACK
- R21 pad 2: /STM32F103 module/DG_FEEDBACK -> /STM32F103 module/POW3_FEEDBACK
- U1 pad 4: /STM32F103 module/DG_FEEDBACK -> /STM32F103 module/POW3_FEEDBACK
- U3 pad 17: (no net) -> /Shutter MOSFET/IN1
- U3 pad 24: /Long stage/SM_CLK -> (no net)
- U3 pad 4: (no net) -> /POW3
- U3 pad 43: /Shutter MOSFET/IN1 -> /Power MOSFET module 2/ON
- U3 pad 45: /Power MOSFET module 2/ON -> (no net)
- U3 pad 46: /POW3 -> (no net)
- U3 pad 55: /Hall8 -> (no net)
- U3 pad 56: /Hall9 -> (no net)
- U3 pad 62: (no net) -> /Long stage/SM_CLK
- U3 pad 92: (no net) -> /Hall8
- U3 pad 93: (no net) -> /Hall9
- U4 pad 5: +3.3V -> +5V
Routing:
- net +5V: track 11.9 -> 429.9 mm, vias 0 -> 5
- net GND: track 112.0 -> 332.6 mm, vias 0 -> 19
- net /Filters slit #1/+24V: track 0.00 -> 194.2 mm
- net /Short stage/SM_EN: track 0.00 -> 161.1 mm, vias 0 -> 2
- net /Short stage/SM_DIR: track 0.00 -> 149.1 mm, vias 0 -> 1
- net /Long stage/SM_EN: track 0.00 -> 140.0 mm, vias 0 -> 2
- net /Long stage/SM_CLK: track 0.00 -> 133.0 mm, vias 0 -> 2
- net /Long stage/SM_DIR: track 0.00 -> 124.1 mm, vias 0 -> 1
- net /Filters slit #2/SM_EN: track 0.00 -> 121.5 mm, vias 0 -> 2
- net /Shutter MOSFET/IN2: track 0.00 -> 112.6 mm, vias 0 -> 2
- net /Shutter MOSFET/IN1: track 0.00 -> 110.2 mm, vias 0 -> 2
- net /Shutter MOSFET/EF: track 0.00 -> 109.0 mm, vias 0 -> 2
- net /Filters slit #1/SM_CLK: track 0.00 -> 106.3 mm, vias 0 -> 4
- net /Filters slit #2/SM_DIR: track 0.00 -> 101.3 mm, vias 0 -> 1
- net /Filters slit #1/SM_EN: track 0.00 -> 97.9 mm, vias 0 -> 2
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- added copper zone on power.Cu, net +3.3V
- added copper zone on power.Cu, net +5V
- added copper zone on power.Cu, net /Filters slit #1/+10V
- added copper zone on ground.Cu, net GND
Other:
- board size 200.5 x 70.9 mm -> 200 x 71 mm
- net class low_power: clearance 0.254 -> 0.1
- board text added: "+10V"
- board text added: "+36V"
- board text added: "+5V"
- board text added: "Filters turret #1"
- board text added: "Filters turret #2"
- board text added: "Focus stage"
- board text added: "Hall sensors"
- board text added: "Master (socket)"
- board text added: "Power load #1"
- board text added: "Power load #2"
- board text added: "Power load (top switch)"
- board text added: "Shutter"
- board text added: "Slave (plug)"
- board text added: "Slits turret"
- board text added: "VPHG stage"
- board text added: "gnd"
- board text removed: "TRD1"

Commit message: last?
Parts:
- removed K1: CONN_3, SIL-3
- removed P1, P14, P18, P19, P8, P9: CONN_2, SIL-2-power
- removed P12: CONN_12, SIL-12
- removed P13: CONN_5, SIL-5
- removed P17, P7: CONN_2, SIL-2
- removed P2, P3, P4, P5, P6: CONN_4, SIL-4-power
- added R40.1: 68, SM1206, B.Cu at (139.3, 128.6)
- added R40.2: 68, SM1206, B.Cu at (161.9, 127.4)
- added XP1: GPRM1-61, gprm1-61, F.Cu at (166.0, 68.5)
- added XP7: Power, VASCH10x2, F.Cu at (175.7, 140.0)
- added hole_3mm: , hole_3mm, F.Cu at (242.0, 67.5)
- added hole_3mm: , hole_3mm, F.Cu at (242.0, 141.5)
- added hole_3mm: , hole_3mm, F.Cu at (48.0, 67.5)
- added hole_3mm: , hole_3mm, F.Cu at (48.0, 141.5)
- added hole_3mm: , hole_3mm, F.Cu at (96.0, 67.5)
- added hole_3mm: , hole_3mm, F.Cu at (135.0, 141.5)
- CON1: footprint MICRO-B-USB -> MINI-B-USB
- DA6: renamed from U5; footprint SOT-223 -> SOT223
- R13, R14, R15, R16: moved to F.Cu
- R19, R27, R28, R29, R30, R31, R32, R33, R34, R37, R38, R39: moved to B.Cu
- XP2: renamed from P10; footprint SIL-8 -> VASCH10x2
- moved R11 61.9 mm to (118.8, 74.1), turned to 180 degrees
- moved R16 45.8 mm to (119.0, 98.5), turned to 270 degrees
- moved VD2 44.0 mm to (78.3, 99.2), turned to 180 degrees
- moved R15 43.7 mm to (122.0, 98.5), turned to 270 degrees
- moved R10 43.6 mm to (78.0, 95.3), turned to 180 degrees
- moved R14 42.2 mm to (125.5, 98.5), turned to 270 degrees
- moved R13 41.5 mm to (129.0, 98.5), turned to 270 degrees
- moved XP4 25.0 mm to (148.4, 143.2)
- moved R38 20.3 mm to (138.4, 131.7), turned to 0 degrees
- moved R37 17.9 mm to (160.3, 131.2)
- moved R25 7.42 mm to (222.8, 140.6), turned to 180 degrees
- moved XS1 7.10 mm to (60.5, 122.5)
- moved XP2 7.07 mm to (113.5, 140.1)
- moved R27 6.74 mm to (104.6, 135.8), turned to 270 degrees
- moved R28 6.74 mm to (107.2, 135.8), turned to 270 degrees
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- renumbered U1 to DA1, U2 to DA2, U4 to DA4, Q3 to DA5, IC1 to DD1, IC2.1 to DD2.1, IC2.2 to DD2.2, IC2.3 to DD2.3, IC2.4 to DD2.4, IC2.5 to DD2.5, U3 to DD3, Q2 to G1, SW1 to SB1, SW2 to SB2, D1 to VD1, D2 to VD2, D3 to VD3, Q1 to VT1, Qp1.1 to VT2.1, Qp1.2 to VT2.2, P11 to XP3, P15 to XP4, P16 to XP5, J2 to XP6, J1 to XS1
Connections:
- DA1 pad 5: N-0000034 -> /POW_LOAD
- DD3 pad 25: /STM32F103 module/RS-232 level converter/UART_TX -> /STM32F103 module/1-WIRE
- DD3 pad 26: /STM32F103 module/RS-232 level converter/UART_RX -> /STM32F103 module/1-WIRE
- DD3 pad 47: /STM32F103 module/1-WIRE -> /STM32F103 module/RS-232 level converter/UART_TX
- DD3 pad 48: /STM32F103 module/1-WIRE -> /STM32F103 module/RS-232 level converter/UART_RX
- DD3 pad 57: /EP0 -> /STM32F103 module/EXT0
- DD3 pad 58: /EP1 -> /STM32F103 module/EXT1
- DD3 pad 59: /EP2 -> /STM32F103 module/EXT2
- DD3 pad 60: /EP3 -> /STM32F103 module/EXT3
- DD3 pad 64: /STM32F103 module/EXT0 -> /EP0
- DD3 pad 65: /STM32F103 module/EXT1 -> /EP1
- DD3 pad 66: /STM32F103 module/EXT2 -> /EP2
- DD3 pad 67: /STM32F103 module/EXT3 -> /EP3
- R11 pad 1: /STM32F103 module/1-WIRE -> +5V
- R11 pad 2: +3.3V -> /STM32F103 module/1-WIRE
- VT2.1 pad 1: /Power MOSFET module 2/ON -> N-00000151
- VT2.2 pad 1: /Power MOSFET module 1/ON -> N-00000126
- XP2 pad 1: /T1_0 -> GND
- XP2 pad 2: /T1_1 -> GND
- XP2 pad 3: /T1_2 -> /T1_0
- XP2 pad 4: /T1_3 -> GND
- XP2 pad 5: /T1_4 -> /T1_1
- XP2 pad 6: /T1_5 -> GND
- XP2 pad 7: /T1_6 -> /T1_2
- XP2 pad 8: /T1_7 -> GND
- XP5 pad 6: /STM32F103 module/RS-232 level converter/UART_TX1 -> /STM32F103 module/RS-232 level converter/UART_RX1
- XP5 pad 7: /STM32F103 module/RS-232 level converter/UART_RX1 -> /STM32F103 module/RS-232 level converter/UART_TX1
Routing:
- net /Shutter MOSFET/+36V: track 5.65 -> 98.7 mm
- net /EP0: track 40.8 -> 88.0 mm
- net /STM32F103 module/1-WIRE: track 30.1 -> 76.2 mm
- net N-0000037: track 4.52 -> 46.2 mm, vias 0 -> 1
- net /Power MOSFET module 2/GND_OUT: track 10.5 -> 51.1 mm, vias 0 -> 1
- net /EP1: track 44.6 -> 82.8 mm
- net /Hall0: track 40.2 -> 75.1 mm
- net /POW_LOAD: track 0.00 -> 34.3 mm
- net /Hall1: track 38.6 -> 72.7 mm
- net /Hall2: track 37.2 -> 69.9 mm
- net /EP2: track 46.4 -> 78.7 mm
- net /Hall3: track 35.6 -> 67.2 mm
- net /Hall4: track 34.9 -> 64.3 mm
- net /Hall5: track 34.2 -> 61.8 mm
- net /EP3: track 48.6 -> 74.6 mm
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- added copper zone on B.Cu, net /Shutter MOSFET/OUT1
- added copper zone on F.Cu, net /Shutter MOSFET/OUT1
- added copper zone on power.Cu, net /Shutter MOSFET/OUT1
- added copper zone on B.Cu, net /Shutter MOSFET/OUT2
- added copper zone on F.Cu, net /Shutter MOSFET/OUT2
- added copper zone on power.Cu, net /Shutter MOSFET/OUT2
Other:
- board size 200 x 71 mm -> 200 x 80 mm
- net class Default: via_dia 0.889 -> 0.9; via_drill 0.635 -> 0.6
- net class low_power: via_dia 0.889 -> 0.9; via_drill 0.635 -> 0.6
- board text added: "+3.3V"
- board text added: "CanRx"
- board text added: "CanTx"
- board text added: "Ext 0..3"
- board text added: "Gnd"
- board text added: "MISO"
- board text added: "MOSI"
- board text added: "SCK"
- board text added: "SCK MISO MOSI"
- board text added: "Tx Rx"
- board text removed: "+10V"
- board text removed: "+36V"
- board text removed: "+5V"
- board text removed: "Filters turret #1"
- board text removed: "Filters turret #2"
- board text removed: "Focus stage"
- board text removed: "Hall sensors"
- board text removed: "Power load #1"
- board text removed: "Power load #2"
- board text removed: "Power load (top switch)"
- board text removed: "Shutter"
- board text removed: "Slits turret"
- board text removed: "VPHG stage"
- board text removed: "gnd"

Commit message: Buttons
Parts:
- R26: moved to B.Cu
- SB1, SB2: footprint SW_PUSH_SMALL -> SPST
- moved R26 20.8 mm to (87.1, 114.9)
- moved SB2 0.65 mm to (72.1, 96.3)
- moved SB1 0.63 mm to (72.0, 106.7)
- moved C7 0.44 mm to (71.8, 112.7)
Routing:
- net GND: track 347.1 -> 338.9 mm
- net /STM32F103 module/BOOT: track 46.7 -> 53.2 mm
- net +3.3V: track 103.1 -> 100.1 mm
- net /STM32F103 module/RST: track 38.9 -> 37.5 mm

Commit message: 1st try to fix errors on PCB
Parts:
- removed hole_3mm (x6): , hole_3mm
- moved XP1 2.45 mm to (167.7, 66.8), turned to 0 degrees
Connections:
- VD1 pad 1: N-0000037 -> N-0000027
- XP1 pad 1-1: /Shutter MOSFET/+36V -> /STM32F103 module/1-WIRE
- XP1 pad 1-11: GND -> /Turret slits/A
- XP1 pad 1-12: GND -> /Turret slits/A*
- XP1 pad 1-13: (no net) -> /Turret slits/B
- XP1 pad 1-14: +5V -> /Turret slits/B*
- XP1 pad 1-15: GND -> /Filters slit #1/A
- XP1 pad 1-16: /EP0 -> /Filters slit #1/A*
- XP1 pad 1-17: /EP1 -> /Filters slit #1/B
- XP1 pad 1-18: /EP2 -> /Filters slit #1/B*
- XP1 pad 1-19: /EP3 -> /Filters slit #2/A
- XP1 pad 1-2: (no net) -> +5V
- XP1 pad 1-20: /Hall0 -> /Filters slit #2/A*
- XP1 pad 1-21: /Hall1 -> /Filters slit #2/B
- XP1 pad 1-22: /Hall2 -> /Filters slit #2/B*
- XP1 pad 1-23: /Hall3 -> /Long stage/A
- XP1 pad 1-24: /Hall4 -> /Long stage/A*
- XP1 pad 1-25: /Hall5 -> /Long stage/B
- XP1 pad 1-26: /Hall6 -> /Long stage/B*
- XP1 pad 1-27: /Hall7 -> /Short stage/A
- XP1 pad 1-28: /Hall8 -> /Short stage/A*
- XP1 pad 1-29: /Hall9 -> /Short stage/B
- XP1 pad 1-3: /Filters slit #1/+10V -> GND
- XP1 pad 1-30: N-0000037 -> /Short stage/B*
- XP1 pad 1-4: /Filters slit #1/+10V -> GND
- XP1 pad 1-5: /Filters slit #1/+10V -> /POW_LOAD
- XP1 pad 1-6: /Filters slit #1/+10V -> /POW_LOAD
- XP1 pad 1-7: (no net) -> GND
- XP1 pad 2-1: /Short stage/B* -> N-0000027
- XP1 pad 2-10: /Filters slit #2/B -> /Hall1
- XP1 pad 2-11: /Filters slit #2/A* -> /Hall0
- XP1 pad 2-12: /Filters slit #2/A -> /EP3
- XP1 pad 2-13: /Filters slit #1/B* -> /EP2
- XP1 pad 2-14: /Filters slit #1/B -> /EP1
- XP1 pad 2-15: /Filters slit #1/A* -> /EP0
- XP1 pad 2-16: /Filters slit #1/A -> GND
- XP1 pad 2-17: /Turret slits/B* -> +5V
- XP1 pad 2-18: /Turret slits/B -> (no net)
- XP1 pad 2-19: /Turret slits/A* -> GND
- XP1 pad 2-2: /Short stage/B -> /Hall9
- XP1 pad 2-20: /Turret slits/A -> GND
- XP1 pad 2-21: (no net) -> GND
- XP1 pad 2-22: (no net) -> GND
- XP1 pad 2-23: (no net) -> GND
- XP1 pad 2-25: /POW_LOAD -> /Filters slit #1/+10V
- XP1 pad 2-26: /POW_LOAD -> /Filters slit #1/+10V
- XP1 pad 2-27: GND -> /Filters slit #1/+10V
- XP1 pad 2-28: GND -> /Filters slit #1/+10V
- XP1 pad 2-29: +5V -> (no net)
- XP1 pad 2-3: /Short stage/A* -> /Hall8
- XP1 pad 2-30: /STM32F103 module/1-WIRE -> /Shutter MOSFET/+36V
- XP1 pad 2-31: GND -> /Shutter MOSFET/+36V
- XP1 pad 2-4: /Short stage/A -> /Hall7
- XP1 pad 2-5: /Long stage/B* -> /Hall6
- XP1 pad 2-6: /Long stage/B -> /Hall5
- XP1 pad 2-7: /Long stage/A* -> /Hall4
- XP1 pad 2-8: /Long stage/A -> /Hall3
- XP1 pad 2-9: /Filters slit #2/B* -> /Hall2
Routing:
- net +5V: track 438.6 -> 381.6 mm
- net (no net): track 0.00 -> 57.0 mm
- net N-0000037: track 46.2 -> 0.00 mm, vias 1 -> 0
- net N-0000027: track 0.00 -> 46.2 mm, vias 0 -> 1
- net /Shutter MOSFET/+36V: track 98.7 -> 102.2 mm

Commit message: modified schematics
Parts:
- added C19: 1u, SM0805, B.Cu at (124.7, 83.3)
- added DA3: RO-1205, SIP-4-RO, F.Cu at (126.7, 86.2)
- added HOLE1: 3mm, hole_3mm, F.Cu at (54.0, 142.0)
- added HOLE2: 3mm, hole_3mm, F.Cu at (54.0, 60.0)
- added HOLE3: 3mm, hole_3mm, F.Cu at (242.0, 142.0)
- added HOLE4: 3mm, hole_3mm, F.Cu at (136.0, 142.0)
- added HOLE5: 3mm, hole_3mm, F.Cu at (242.0, 60.0)
- added HOLE6: 3mm, hole_3mm, F.Cu at (98.0, 60.0)
- added P1: CONN_1, PIN_ARRAY_1, F.Cu at (237.5, 118.5)
- added P2: CONN_1, PIN_ARRAY_1, F.Cu at (97.8, 79.2)
- added R41: 56k, SM0603, F.Cu at (180.7, 126.0)
- added R42: 4.7k, SM0603, F.Cu at (180.7, 128.0)
- added R43: 12k, SM0603, B.Cu at (90.3, 126.4)
- added R44: 4.7k, SM0603, F.Cu at (91.8, 122.2)
- added U1: LM7805CT, TO220_VERT, F.Cu at (129.4, 82.4)
- R1.1, R1.2, R1.3, R1.4, R1.5, R2.1, R2.2, R2.3, R2.4, R2.5: footprint SM1210 -> SM-2010
- VT2.1, VT2.2: value NTE2984 -> FQP30N06
- XP6: value DB9 -> DB9-M; footprint DB9FC -> DB9-M
- XS1: value DB9 -> DB9-F; footprint DB9FC -> DB9-F
- moved C14 15.4 mm to (98.2, 134.2), turned to 180 degrees
- moved CON1 7.50 mm to (85.8, 62.9)
- moved XP6 5.77 mm to (60.5, 81.0)
- moved R38 3.68 mm to (142.1, 131.7)
- moved R40.1 3.68 mm to (143.0, 128.6)
- moved R2.5 3.46 mm to (237.6, 110.9), turned to 90 degrees
- moved R2.4 3.44 mm to (215.6, 110.9), turned to 90 degrees
- moved R2.2 3.04 mm to (170.9, 110.6), turned to 90 degrees
- moved R1.1 3.04 mm to (150.2, 86.7), turned to 270 degrees
- moved R2.1 3.00 mm to (150.0, 110.5), turned to 90 degrees
- moved R1.2 2.97 mm to (170.9, 87.0), turned to 270 degrees
- moved R1.4 2.95 mm to (216.2, 86.9), turned to 270 degrees
- moved R2.3 2.93 mm to (193.7, 110.5), turned to 90 degrees
- moved R1.3 2.87 mm to (193.9, 87.0), turned to 270 degrees
- moved R1.5 2.86 mm to (238.3, 87.0), turned to 270 degrees
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Connections:
- DA5 pad 1: /Filters slit #1/+10V -> GND
- DA5 pad 2: GND -> /Filters slit #1/+10V
- DA5 pad 3: /Filters slit #1/+24V -> GND
- DA5 pad 4: GND -> /Filters slit #1/+24V
- DD1 pad 18: N-00000157 -> N-00000155
- DD3 pad 23: (no net) -> /STM32F103 module/U10
- DD3 pad 24: (no net) -> /Shutter MOSFET/Sense
- VT1 pad 2: +5V -> +3.3V
- XP6 pad 2: N-00000157 -> N-00000169
- XP6 pad 3: N-00000169 -> N-00000155
Routing:
- net /Shutter MOSFET/Sense: track 0.00 -> 102.7 mm, vias 0 -> 2
- net N-00000155: track 0.00 -> 79.3 mm
- net /Filters slit #1/+10V: track 41.4 -> 119.7 mm, vias 0 -> 1
- net +5V: track 381.6 -> 453.3 mm, vias 5 -> 4
- net N-00000157: track 70.4 -> 0.00 mm
- net (no net): track 57.0 -> 0.00 mm
- net GND: track 338.9 -> 309.3 mm, vias 20 -> 23
- net +3.3V: track 100.1 -> 111.7 mm, vias 14 -> 15
- net N-00000175: track 13.5 -> 22.2 mm
- net N-00000169: track 74.9 -> 83.3 mm
- net /STM32F103 module/U10: track 0.00 -> 8.46 mm, vias 0 -> 1
- net N-00000171: track 10.2 -> 17.7 mm
- net N-00000170: track 10.6 -> 18.1 mm
- net /EP3: track 74.6 -> 81.7 mm
- net N-00000147: track 43.1 -> 49.0 mm
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Other:
- board size 200 x 80 mm -> 194 x 88 mm
- board text added: "+24V"
- board text added: "+5V"
- board text added: "3RC = 0.66s"
