File: schematic/ALL.kicad_pcb (KiCad board)
At the start: 4 copper layers, 194 x 88 mm, 141 parts, among them CON1 USB-MICRO-B, P1 CONN_1, P2 CONN_1, U1 LM7805CT

Commit message: save under new kicad
Parts:
- removed C19: 1u, SM0805
- removed DA3: RO-1205, SIP-4-RO
- removed HOLE1, HOLE2, HOLE3, HOLE4, HOLE5, HOLE6: 3mm, hole_3mm
- removed R40.1, R40.2: 68, SM1206
- removed R41: 56k, SM0603
- removed R42, R44: 4.7k, SM0603
- removed R43: 12k, SM0603
- removed the U1 at (129.4, 82.4)
- removed XP1: GPRM1-61, gprm1-61
- removed XP6: DB9-M, DB9-M
- removed XP7: Power, VASCH10x2
- added J2: DB9, DB9FC, F.Cu at (60.5, 91.0)
- added K1: CONN_3, SIL-3, F.Cu at (92.1, 143.5)
- added P12: CONN_12, SIL-12, F.Cu at (105.8, 75.8)
- added P13: CONN_5, SIL-5, F.Cu at (137.1, 143.5)
- added P14: CONN_2, SIL-2-power, F.Cu at (226.2, 193.7)
- added P17: CONN_2, SIL-2, F.Cu at (89.2, 128.0)
- added P18: CONN_2, SIL-2-power, F.Cu at (126.2, 191.8)
- added P19: CONN_2, SIL-2-power, F.Cu at (246.5, 180.2)
- added P3: CONN_4, SIL-4-power, F.Cu at (207.1, 77.3)
- added P4: CONN_4, SIL-4-power, F.Cu at (228.7, 77.2)
- added P5: CONN_4, SIL-4-power, F.Cu at (162.4, 77.5)
- added P6: CONN_4, SIL-4-power, F.Cu at (185.1, 77.3)
- added P7: CONN_2, SIL-2, F.Cu at (69.8, 75.8)
- added P8: CONN_2, SIL-2-power, F.Cu at (180.2, 175.5)
- added P9: CONN_2, SIL-2-power, F.Cu at (154.3, 172.2)
- CON1: footprint MINI-B-USB -> MICRO-B-USB
- J1: renamed from XS1; value DB9-F -> DB9; footprint DB9-F -> DB9FC
- P1: value CONN_1 -> CONN_2; footprint PIN_ARRAY_1 -> SIL-2-power
- P10: renamed from XP2; footprint VASCH10x2 -> SIL-8
- P2: value CONN_1 -> CONN_4; footprint PIN_ARRAY_1 -> SIL-4-power
- Qp1.1: renamed from VT2.1; value FQP30N06 -> NTE2984
- Qp1.2: renamed from VT2.2; value FQP30N06 -> NTE2984
- R1.1, R1.2, R1.3, R1.4, R1.5, R2.1, R2.2, R2.3, R2.4, R2.5: footprint SM-2010 -> SM1210
- R11, R19, R22, R23, R24, R26, R27, R28, R29, R30, R31, R32, R33, R34, R37, R38, R39: moved to F.Cu
- R13, R14, R15, R16: moved to B.Cu
- R25: value 300 (II) -> 1.2k (II)
- SW1: renamed from SB1; footprint SPST -> SW_PUSH_SMALL
- SW2: renamed from SB2; footprint SPST -> SW_PUSH_SMALL
- U5: renamed from DA6; footprint SOT223 -> SOT-223
- moved R23 123.1 mm to (224.3, 182.8), turned to 180 degrees
- moved R24 113.6 mm to (224.7, 180.2), turned to 180 degrees
- moved R22 107.2 mm to (209.3, 187.3)
- moved R39 97.7 mm to (118.4, 180.3), turned to 180 degrees
- moved U1 95.1 mm to (127.2, 181.0)
- moved R20 90.3 mm to (120.4, 183.5), turned to 270 degrees
- moved R11 72.6 mm to (91.3, 141.3)
- moved U2 58.5 mm to (217.3, 181.5), turned to 0 degrees
- moved R16 45.8 mm to (138.3, 140.0), turned to 90 degrees
- moved D2 44.0 mm to (120.7, 110.7), turned to 270 degrees
- moved R15 43.7 mm to (135.8, 140.0), turned to 90 degrees
- moved R10 43.6 mm to (118.4, 111.8), turned to 0 degrees
- moved P2 43.4 mm to (141.1, 77.4)
- moved R19 43.3 mm to (109.6, 128.1)
- moved Q3 42.7 mm to (196.7, 130.2)
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- renumbered VD1 to D1, VD2 to D2, VD3 to D3, DD1 to IC1, DD2.1 to IC2.1, DD2.2 to IC2.2, DD2.3 to IC2.3, DD2.4 to IC2.4, DD2.5 to IC2.5, XP3 to P11, XP4 to P15, XP5 to P16, VT1 to Q1, G1 to Q2, DA5 to Q3, DA1 to U1, DA2 to U2, DD3 to U3, DA4 to U4
Connections:
- net /STM32F103 module/POW3_FEEDBACK renamed /STM32F103 module/SHTR_FEEDBACK
- C12 pad 2: +5V -> +3.3V
- P1 pad 1: /Filters slit #1/+24V -> GND
- P10 pad 1: GND -> /T1_0
- P10 pad 2: GND -> /T1_1
- P10 pad 3: /T1_0 -> /T1_2
- P10 pad 4: GND -> /T1_3
- P10 pad 5: /T1_1 -> /T1_4
- P10 pad 6: GND -> /T1_5
- P10 pad 7: /T1_2 -> /T1_6
- P10 pad 8: GND -> /T1_7
- P16 pad 6: /STM32F103 module/RS-232 level converter/UART_RX1 -> /STM32F103 module/RS-232 level converter/UART_TX1
- P16 pad 7: /STM32F103 module/RS-232 level converter/UART_TX1 -> /STM32F103 module/RS-232 level converter/UART_RX1
- P2 pad 1: +5V -> /Turret slits/A
- Q3 pad 1: GND -> /Filters slit #1/+10V
- Q3 pad 2: /Filters slit #1/+10V -> GND
- Q3 pad 3: GND -> /Filters slit #1/+24V
- Q3 pad 4: /Filters slit #1/+24V -> GND
- Qp1.1 pad 1: N-00000146 (its old number) -> /Power MOSFET module 2/ON
- Qp1.2 pad 1: N-00000121 (its old number) -> /Power MOSFET module 1/ON
- R11 pad 1: +5V -> /STM32F103 module/1-WIRE
- R11 pad 2: /STM32F103 module/1-WIRE -> +3.3V
- R13 pad 2: +3.3V -> +5V
- R14 pad 2: +3.3V -> +5V
- R15 pad 2: +3.3V -> +5V
- R16 pad 2: +3.3V -> +5V
- U1 pad 5: /POW_LOAD -> N-0000034
- U3 pad 17: /Shutter MOSFET/IN1 -> (no net)
- U3 pad 23: /STM32F103 module/U10 -> (no net)
- U3 pad 24: /Shutter MOSFET/Sense -> /Long stage/SM_CLK
- U3 pad 25: /STM32F103 module/1-WIRE -> /STM32F103 module/RS-232 level converter/UART_TX
- U3 pad 26: /STM32F103 module/1-WIRE -> /STM32F103 module/RS-232 level converter/UART_RX
- U3 pad 4: /POW3 -> (no net)
- U3 pad 43: /Power MOSFET module 2/ON -> /Shutter MOSFET/IN1
- U3 pad 45: (no net) -> /Power MOSFET module 2/ON
- U3 pad 46: (no net) -> /POW3
- U3 pad 47: /STM32F103 module/RS-232 level converter/UART_TX -> /STM32F103 module/1-WIRE
- U3 pad 48: /STM32F103 module/RS-232 level converter/UART_RX -> /STM32F103 module/1-WIRE
- U3 pad 55: (no net) -> /Hall8
- U3 pad 56: (no net) -> /Hall9
- U3 pad 57: /STM32F103 module/EXT0 -> /EP0
- U3 pad 58: /STM32F103 module/EXT1 -> /EP1
- U3 pad 59: /STM32F103 module/EXT2 -> /EP2
- U3 pad 60: /STM32F103 module/EXT3 -> /EP3
- U3 pad 62: /Long stage/SM_CLK -> (no net)
- U3 pad 64: /EP0 -> /STM32F103 module/EXT0
- U3 pad 65: /EP1 -> /STM32F103 module/EXT1
- U3 pad 66: /EP2 -> /STM32F103 module/EXT2
- U3 pad 67: /EP3 -> /STM32F103 module/EXT3
- U3 pad 92: /Hall8 -> (no net)
- U3 pad 93: /Hall9 -> (no net)
- U4 pad 5: +5V -> +3.3V
Routing:
- net +5V: track 453.3 -> 11.9 mm, vias 4 -> 0
- net /Filters slit #1/+24V: track 208.7 -> 0.00 mm, vias 2 -> 0
- net GND: track 309.3 -> 112.0 mm, vias 23 -> 0
- net /Short stage/SM_EN: track 160.5 -> 0.00 mm, vias 2 -> 0
- net /Short stage/SM_DIR: track 150.5 -> 0.00 mm, vias 1 -> 0
- net /Long stage/SM_EN: track 139.6 -> 0.00 mm, vias 2 -> 0
- net /Long stage/SM_CLK: track 133.0 -> 0.00 mm, vias 2 -> 0
- net /Long stage/SM_DIR: track 125.2 -> 0.00 mm, vias 1 -> 0
- net /Filters slit #2/SM_EN: track 121.2 -> 0.00 mm, vias 2 -> 0
- net /Filters slit #1/+10V: track 119.7 -> 0.00 mm, vias 1 -> 0
- net /Shutter MOSFET/IN2: track 114.8 -> 0.00 mm, vias 2 -> 0
- net /Shutter MOSFET/EF: track 111.2 -> 0.00 mm, vias 2 -> 0
- net /Shutter MOSFET/IN1: track 109.5 -> 0.00 mm, vias 2 -> 0
- net /Filters slit #1/SM_CLK: track 106.3 -> 0.00 mm, vias 4 -> 0
- net /Shutter MOSFET/+36V: track 104.5 -> 0.00 mm
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- removed copper zone on power.Cu, net +3.3V
- removed copper zone on power.Cu, net +5V
- removed copper zone on power.Cu, net /Filters slit #1/+10V
- removed copper zone on B.Cu, net /Shutter MOSFET/OUT1
- removed copper zone on F.Cu, net /Shutter MOSFET/OUT1
- removed copper zone on power.Cu, net /Shutter MOSFET/OUT1
- removed copper zone on B.Cu, net /Shutter MOSFET/OUT2
- removed copper zone on F.Cu, net /Shutter MOSFET/OUT2
- removed copper zone on power.Cu, net /Shutter MOSFET/OUT2
- removed copper zone on ground.Cu, net GND
Other:
- board size 194 x 88 mm -> 200.5 x 70.9 mm
- net class Default: via_dia 0.9 -> 0.889; via_drill 0.6 -> 0.635
- net class low_power: clearance 0.1 -> 0.254; via_dia 0.9 -> 0.889; via_drill 0.6 -> 0.635
- board text added: "TRD1"
- board text removed: "+24V"
- board text removed: "+3.3V"
- board text removed: "+5V"
- board text removed: "3RC = 0.66s"
- board text removed: "CanRx"
- board text removed: "CanTx"
- board text removed: "Ext 0..3"
- board text removed: "Gnd"
- board text removed: "MISO"
- board text removed: "MOSI"
- board text removed: "Master (socket)"
- board text removed: "SCK"
- board text removed: "SCK MISO MOSI"
- board text removed: "Slave (plug)"
- board text removed: "Tx Rx"
