File: schematic/ALL.sch (KiCad schematic (older format))
At the start: 20 parts, among them K1 CONN_3, P1 CONN_2, P10 TRD, P12 CONN_12, P13 CONN_5, P14 CONN_2, P18 CONN_2, P19 CONN_2, P2 CONN_4, P3 CONN_4, P4 CONN_4, P5 CONN_4, P6 CONN_4, P7 CONN_2, P8 CONN_2, P9 CONN_2, Q3 RO-1224, U1 IPS5451

Commit message: PCB
Connections:
- net STM32F103 module/SHTR_FEEDBACK renamed STM32F103 module/POW3_FEEDBACK
Changed lines of the file:
@@
-EESchema Schematic File Version 2  date Ср 09 июл 2014 18:42:33
+EESchema Schematic File Version 2  date Пт 11 июл 2014 12:31:03
 LIBS:power
 LIBS:device
@@
 Sheet 1 12
 Title "IR-spectrometer Control System"
-Date "9 jul 2014"
+Date "11 jul 2014"
 Rev ""
 Comp "SAO RAS"
@@
 F11 "POW[0..3]" O L 6300 6050 60
 F12 "ADC[0..7]" I R 8100 2750 60
-F13 "SHTR_FEEDBACK" I L 6300 6600 60
+F13 "POW3_FEEDBACK" I L 6300 6600 60
 F14 "SHTR" O L 6300 6250 60
 F15 "SHTR_FB" I L 6300 6400 60

Commit message: last?
Parts:
- removed K1: CONN_3, SIL-3, symbol CONN_3
- removed P1, P14, P18, P19, P8, P9: CONN_2, SIL-2-power, symbol CONN_2
- removed P12: CONN_12, SIL-12, symbol CONN_12
- removed P13: CONN_5, SIL-5, symbol CONN_5
- removed P2, P3, P4, P5, P6: CONN_4, SIL-4-power, symbol CONN_4
- removed P7: CONN_2, SIL-2, symbol CONN_2
- added XP1: GPRM1-61, gprm1-61, symbol GPRM1-61
- added XP7: Power, VASCH10x2, symbol CONN_10X2
- XP2: renamed from P10; footprint SIL-8 -> VASCH10x2; symbol CONN_8 -> CONN_10X2
- renumbered U1 to DA1, Q3 to DA5, D1 to VD1
Connections:
- net labels added: 1-wire, 1A, 1B, 1C, 1D, 2A, 2B, 2C, 2D, 3A, 3B, 3C, 3D, 4A, 4B, 4C, 4D, 5A, 5B, 5C, 5D, POW_GND1, POW_GND2, POW_LOAD, Shutter1, Shutter2
- wire segments 190 -> 227
- no-connect marks 0 -> 11
Other:
- note added: "5V ext"
- note added: "5V out"
- note added: "End point\nswitches"
- note added: "Power ground"
- note added: "Power load\n(bottom switches)"
- note added: "Power load\n(top switch)"
- note added: "Power sources:\n36V - 300mA\n10V - 7.5A\n5V - 0.5A"
- note added: "Shutter control"
- note added: "Shutter out"
- note added: "Signal ground"
- note added: "Stepper"
- note added: "To thermoresistors"
- note removed: "1-wire"
- note removed: "10V"
- note removed: "36V"
- note removed: "5V"
- note removed: "Power load (bottom switch)"
- note removed: "Power load (top switch)"
- note removed: "Shutter"
- note removed: "К терморезисторам"
- moved on the sheet: VD1

Commit message: 1st try to fix errors on PCB
Connections:
- wire segments 227 -> 230
- no-connect marks 11 -> 7
Changed lines of the file:
@@
-EESchema Schematic File Version 2  date Пн 21 июл 2014 09:59:08
+EESchema Schematic File Version 2  date Пн 29 сен 2014 14:40:29
 LIBS:power
 LIBS:device
@@
 Sheet 1 12
 Title "IR-spectrometer Control System"
-Date "21 jul 2014"
+Date "29 sep 2014"
 Rev ""
 Comp "SAO RAS"
@@
 Text Notes 3550 3200 0    60   ~ 0
 5V out
-$Comp
-L GPRM1-61 XP1
-U 1 1 53DA1715
-P 2850 3350
-F 0 "XP1" H 2850 1650 50  0000 C CNN
-F 1 "GPRM1-61" V 2850 3350 50  0000 C CNN
-F 2 "gprm1-61" H 2850 3350 50  0001 C CNN
-F 3 "~" H 2850 3350 50  0001 C CNN
-	1    2850 3350
-	-1   0    0    -1
-$EndComp
 Text Notes 4300 3450 0    61   ~ 0
 End point\nswitches
@@
 L GNDPWR #PWR028
 U 1 1 53DFE593
-P 2400 5050
-F 0 "#PWR028" H 2400 5100 40  0001 C CNN
-F 1 "GNDPWR" H 2400 4970 40  0000 C CNN
-F 2 "" H 2400 5050 60  0000 C CNN
-F 3 "" H 2400 5050 60  0000 C CNN
-	1    2400 5050
-	1    0    0    -1
-$EndComp
-Wire Wire Line
-	2400 5050 2400 4850
+P 1750 4100
+F 0 "#PWR028" H 1750 4150 40  0001 C CNN
+F 1 "GNDPWR" H 1750 4020 40  0000 C CNN
+F 2 "" H 1750 4100 60  0000 C CNN
+F 3 "" H 1750 4100 60  0000 C CNN
+	1    1750 4100
+	1    0    0    -1
+$EndComp
 Wire Wire Line
 	2400 4650 1800 4650
@@
 Connection ~ 1600 6750
 Connection ~ 1600 6550
-NoConn ~ 2400 4150
-NoConn ~ 2400 4050
-NoConn ~ 2400 3950
-NoConn ~ 2400 3850
 NoConn ~ 1900 6350
 NoConn ~ 2700 6350
@@
 Wire Wire Line
 	2400 4350 1600 4350
+Wire Wire Line
+	1750 4000 1750 4100
+$Comp
+L GPRM1-61 XP1
+U 1 1 53DA1715
+P 2850 3300
+F 0 "XP1" H 2850 1600 50  0000 C CNN
+F 1 "GPRM1-61" V 2850 3300 50  0000 C CNN
+F 2 "gprm1-61" H 2850 3300 50  0001 C CNN
+F 3 "~" H 2850 3300 50  0001 C CNN
+	1    2850 3300
+	1    0    0    1
+$EndComp
+Wire Wire Line
+	2400 4150 2400 3850
+Wire Wire Line
+	1750 4000 2400 4000
+Connection ~ 2400 4000
+Connection ~ 2400 4050
+Connection ~ 2400 3950
+Wire Wire Line
+	3300 1800 3300 1900
+Connection ~ 3300 1900
 $EndSCHEMATC

Commit message: modified schematics
Parts:
- added C19: 1u, SM0805, symbol C
- added DA3: RO-1205, SIP-4-RO, symbol RO-XX
- added HOLE1, HOLE2, HOLE3, HOLE4, HOLE5, HOLE6: 3mm, symbol HOLE
- added P1, P2: CONN_1, symbol CONN_1
- added R43: 12k, SM0603, symbol R0603
- added R44: 4.7k, SM0603, symbol R0603
- added U1: LM7805CT, TO-220, symbol LM7805CT
Connections:
- wire segments 230 -> 249
Other:
- note added: "Place DA3 OR U1"
- note added: "TEST24"
- note added: "TEST5"
