File: schematic/MCU_module.sch (KiCad schematic (older format))
At the start: 49 parts, among them P11 CONN_7, P15 CONN_4, P16 CONN_7, Q2 8MHz, SW1 RESET, SW2 BOOT, U3 STM32F103, U5 LM1117MPX-3.3

Commit message: PCB
Connections:
- net labels added: POW3_FEEDBACK
- net labels removed: SHTR_FEEDBACK
- wire segments 206 -> 200

Commit message: last?
Parts:
- renumbered U5 to DA6, U3 to DD3, Q2 to G1, SW1 to SB1, SW2 to SB2, D2 to VD2, P11 to XP3, P15 to XP4, P16 to XP5
Connections:
- net labels added: AGND
- wire segments 200 -> 202
Other:
- moved on the sheet: R11

Commit message: Buttons
Parts:
- SB1, SB2: footprint SW_PUSH_SMALL -> SPST
Changed lines of the file:
@@
-EESchema Schematic File Version 2  date Пт 18 июл 2014 12:36:52
+EESchema Schematic File Version 2  date Пн 21 июл 2014 09:59:08
 LIBS:power
 LIBS:device
@@
 Sheet 3 12
 Title "MCU module on STM32F103"
-Date "18 jul 2014"
+Date "21 jul 2014"
 Rev ""
 Comp "SAO RAS"
@@
 F 0 "SB1" H 8100 1160 50  0000 C CNN
 F 1 "RESET" H 7950 970 50  0000 C CNN
-F 2 "SW_PUSH_SMALL" H 7950 1050 60  0001 C CNN
+F 2 "SPST" H 7950 1050 60  0001 C CNN
 F 3 "~" H 7950 1050 60  0000 C CNN
 	1    7950 1050
@@
 F 0 "SB2" H 9350 1160 50  0000 C CNN
 F 1 "BOOT" H 9200 970 50  0000 C CNN
-F 2 "SW_PUSH_SMALL" H 9200 1050 60  0001 C CNN
+F 2 "SPST" H 9200 1050 60  0001 C CNN
 F 3 "~" H 9200 1050 60  0000 C CNN
 	1    9200 1050

Commit message: modified schematics
Connections:
- net labels added: U10, U10_ADC, U36, U36_ADC
- wire segments 202 -> 204
- no-connect marks 19 -> 17
Changed lines of the file:
@@
-EESchema Schematic File Version 2  date Вт 07 окт 2014 17:18:47
+EESchema Schematic File Version 2  date Вс 30 ноя 2014 15:36:58
 LIBS:power
 LIBS:device
@@
 Sheet 3 12
 Title "MCU module on STM32F103"
-Date "7 oct 2014"
+Date "30 nov 2014"
 Rev ""
 Comp "SAO RAS"
@@
 $EndDescr
 $Comp
-L GND #PWR040
+L GND #PWR043
 U 1 1 5396087F
 P 800 10900
-F 0 "#PWR040" H 800 10900 30  0001 C CNN
+F 0 "#PWR043" H 800 10900 30  0001 C CNN
 F 1 "GND" H 800 10830 30  0001 C CNN
 F 2 "" H 800 10900 60  0000 C CNN
@@
 USB_DM
 NoConn ~ 15300 5600
-NoConn ~ 8300 7600
 NoConn ~ 8300 6000
 NoConn ~ 8300 5900
@@
 $EndComp
 $Comp
-L +3.3V #PWR041
+L +3.3V #PWR044
 U 1 1 5396A0D9
 P 13300 9100
-F 0 "#PWR041" H 13300 9060 30  0001 C CNN
+F 0 "#PWR044" H 13300 9060 30  0001 C CNN
 F 1 "+3.3V" H 13300 9210 30  0000 C CNN
 F 2 "" H 13300 9100 60  0000 C CNN
@@
 $EndComp
 $Comp
-L GND #PWR042
+L GND #PWR045
 U 1 1 5396A64A
 P 12900 9400
-F 0 "#PWR042" H 12900 9400 30  0001 C CNN
+F 0 "#PWR045" H 12900 9400 30  0001 C CNN
 F 1 "GND" H 12900 9330 30  0001 C CNN
 F 2 "" H 12900 9400 60  0000 C CNN
@@
 $EndComp
 $Comp
-L GND #PWR043
+L GND #PWR046
 U 1 1 5396ADE7
 P 7500 6250
-F 0 "#PWR043" H 7500 6250 30  0001 C CNN
+F 0 "#PWR046" H 7500 6250 30  0001 C CNN
 F 1 "GND" H 7500 6180 30  0001 C CNN
 F 2 "" H 7500 6250 60  0000 C CNN
@@
 $EndComp
 $Comp
-L +3.3V #PWR044
+L +3.3V #PWR047
 U 1 1 5396AE12
 P 7800 6450
-F 0 "#PWR044" H 7800 6410 30  0001 C CNN
+F 0 "#PWR047" H 7800 6410 30  0001 C CNN
 F 1 "+3.3V" H 7800 6560 30  0000 C CNN
 F 2 "" H 7800 6450 60  0000 C CNN
@@
 $EndComp
 $Comp
-L GND #PWR045
+L GND #PWR048
 U 1 1 5396C0F4
 P 15700 5500
-F 0 "#PWR045" H 15700 5500 30  0001 C CNN
+F 0 "#PWR048" H 15700 5500 30  0001 C CNN
 F 1 "GND" H 15700 5430 30  0001 C CNN
 F 2 "" H 15700 5500 60  0000 C CNN
@@
 $EndComp
 $Comp
-L +3.3V #PWR046
+L +3.3V #PWR049
 U 1 1 5396C0FB
 P 15300 5100
-F 0 "#PWR046" H 15300 5060 30  0001 C CNN
+F 0 "#PWR049" H 15300 5060 30  0001 C CNN
 F 1 "+3.3V" H 15300 5210 30  0000 C CNN
 F 2 "" H 15300 5100 60  0000 C CNN
@@
 $EndComp
 $Comp
-L +3.3V #PWR047
+L +3.3V #PWR050
 U 1 1 5396C797
 P 10300 4100
-F 0 "#PWR047" H 10300 4060 30  0001 C CNN
+F 0 "#PWR050" H 10300 4060 30  0001 C CNN
 F 1 "+3.3V" H 10300 4210 30  0000 C CNN
 F 2 "" H 10300 4100 60  0000 C CNN
@@
 $EndComp
 $Comp
-L GND #PWR048
+L GND #PWR051
 U 1 1 5396CC1B
 P 10600 3950
-F 0 "#PWR048" H 10600 3950 30  0001 C CNN
+F 0 "#PWR051" H 10600 3950 30  0001 C CNN
 F 1 "GND" H 10600 3880 30  0001 C CNN
 F 2 "" H 10600 3950 60  0000 C CNN
@@
 $EndComp
 $Comp
-L GND #PWR049
+L GND #PWR052
 U 1 1 539753BB
 P 6850 1350
-F 0 "#PWR049" H 6850 1350 30  0001 C CNN
+F 0 "#PWR052" H 6850 1350 30  0001 C CNN
 F 1 "GND" H 6850 1280 30  0001 C CNN
 F 2 "" H 6850 1350 60  0000 C CNN
@@
 +5V
 $Comp
-L GND #PWR050
+L GND #PWR053
 U 1 1 5397CF1C
 P 4100 1250
-F 0 "#PWR050" H 4100 1250 30  0001 C CNN
+F 0 "#PWR053" H 4100 1250 30  0001 C CNN
 F 1 "GND" H 4100 1180 30  0001 C CNN
 F 2 "" H 4100 1250 60  0000 C CNN
@@
 GND
 $Comp
-L +5V #PWR051
+L +5V #PWR054
 U 1 1 53994516
 P 4400 650
-F 0 "#PWR051" H 4400 740 20  0001 C CNN
+F 0 "#PWR054" H 4400 740 20  0001 C CNN
 F 1 "+5V" H 4400 740 30  0000 C CNN
 F 2 "" H 4400 650 60  0000 C CNN
@@
 $EndComp
 $Comp
-L GND #PWR052
+L GND #PWR055
 U 1 1 5399714A
 P 4900 1450
-F 0 "#PWR052" H 4900 1450 30  0001 C CNN
+F 0 "#PWR055" H 4900 1450 30  0001 C CNN
 F 1 "GND" H 4900 1380 30  0001 C CNN
 F 2 "" H 4900 1450 60  0000 C CNN
@@
 $EndComp
 $Comp
-L +3.3V #PWR053
+L +3.3V #PWR056
 U 1 1 5399760C
 P 5450 650
-F 0 "#PWR053" H 5450 610 30  0001 C CNN
+F 0 "#PWR056" H 5450 610 30  0001 C CNN
 F 1 "+3.3V" H 5450 760 30  0000 C CNN
 F 2 "" H 5450 650 60  0000 C CNN
@@
 $EndComp
 $Comp
-L GND #PWR054
+L GND #PWR057
 U 1 1 5399B981
 P 8150 1450
-F 0 "#PWR054" H 8150 1450 30  0001 C CNN
+F 0 "#PWR057" H 8150 1450 30  0001 C CNN
 F 1 "GND" H 8150 1380 30  0001 C CNN
 F 2 "" H 8150 1450 60  0000 C CNN
@@
 $EndComp
 $Comp
-L +3.3V #PWR055
+L +3.3V #PWR058
 U 1 1 5399BA1F
 P 7600 1450
-F 0 "#PWR055" H 7600 1410 30  0001 C CNN
+F 0 "#PWR058" H 7600 1410 30  0001 C CNN
 F 1 "+3.3V" H 7600 1560 30  0000 C CNN
 F 2 "" H 7600 1450 60  0000 C CNN
@@
 $EndComp
 $Comp
-L +3.3V #PWR056
+L +3.3V #PWR059
 U 1 1 539ADE4F
 P 1950 1150
-F 0 "#PWR056" H 1950 1110 30  0001 C CNN
+F 0 "#PWR059" H 1950 1110 30  0001 C CNN
 F 1 "+3.3V" H 1950 1260 30  0000 C CNN
 F 2 "" H 1950 1150 60  0000 C CNN
@@
 $EndComp
 $Comp
-L PWR_FLAG #FLG057
+L PWR_FLAG #FLG060
 U 1 1 539B6CB5
 P 6850 900
-F 0 "#FLG057" H 6850 995 30  0001 C CNN
+F 0 "#FLG060" H 6850 995 30  0001 C CNN
 F 1 "PWR_FLAG" H 6850 1080 30  0000 C CNN
 F 2 "" H 6850 900 60  0000 C CNN
@@
 $EndComp
 $Comp
-L GND #PWR058
+L GND #PWR061
 U 1 1 539789E9
 P 3150 10550
-F 0 "#PWR058" H 3150 10550 30  0001 C CNN
+F 0 "#PWR061" H 3150 10550 30  0001 C CNN
 F 1 "GND" H 3150 10480 30  0001 C CNN
 F 2 "" H 3150 10550 60  0000 C CNN
@@
 Power
 $Comp
-L +5V #PWR059
+L +5V #PWR062
 U 1 1 539BABDD
 P 600 10350
-F 0 "#PWR059" H 600 10440 20  0001 C CNN
+F 0 "#PWR062" H 600 10440 20  0001 C CNN
 F 1 "+5V" H 600 10440 30  0000 C CNN
 F 2 "" H 600 10350 60  0000 C CNN
@@
 $EndComp
 $Comp
-L GND #PWR060
+L GND #PWR063
 U 1 1 53A797DF
 P 10500 9250
-F 0 "#PWR060" H 10500 9250 30  0001 C CNN
+F 0 "#PWR063" H 10500 9250 30  0001 C CNN
 F 1 "GND" H 10500 9180 30  0001 C CNN
 F 2 "" H 10500 9250 60  0000 C CNN
@@
 $EndComp
 $Comp
-L +3.3V #PWR061
+L +3.3V #PWR064
 U 1 1 53A79926
 P 10800 9700
-F 0 "#PWR061" H 10800 9660 30  0001 C CNN
+F 0 "#PWR064" H 10800 9660 30  0001 C CNN
 F 1 "+3.3V" H 10800 9810 30  0000 C CNN
 F 2 "" H 10800 9700 60  0000 C CNN
@@
 $EndComp
 $Comp
-L GND #PWR062
+L GND #PWR065
 U 1 1 53B31F80
 P 6300 6800
-F 0 "#PWR062" H 6300 6800 30  0001 C CNN
+F 0 "#PWR065" H 6300 6800 30  0001 C CNN
 F 1 "GND" H 6300 6730 30  0001 C CNN
 F 2 "" H 6300 6800 60  0000 C CNN
@@
 $EndComp
 $Comp
-L GND #PWR063
+L GND #PWR066
 U 1 1 53A25FC1
 P 4550 2700
-F 0 "#PWR063" H 4550 2700 30  0001 C CNN
+F 0 "#PWR066" H 4550 2700 30  0001 C CNN
 F 1 "GND" H 4550 2630 30  0001 C CNN
 F 2 "" H 4550 2700 60  0000 C CNN
@@
 Additional IO
 $Comp
-L GND #PWR064
+L GND #PWR067
 U 1 1 53A3632D
 P 4750 4400
-F 0 "#PWR064" H 4750 4400 30  0001 C CNN
+F 0 "#PWR067" H 4750 4400 30  0001 C CNN
 F 1 "GND" H 4750 4330 30  0001 C CNN
 F 2 "" H 4750 4400 60  0000 C CNN
@@
 $EndComp
 $Comp
-L GND #PWR065
+L GND #PWR068
 U 1 1 53A3CC3C
 P 11700 9950
-F 0 "#PWR065" H 11700 9950 30  0001 C CNN
+F 0 "#PWR068" H 11700 9950 30  0001 C CNN
 F 1 "GND" H 11700 9880 30  0001 C CNN
 F 2 "" H 11700 9950 60  0000 C CNN
@@
 $EndComp
 $Comp
-L GND #PWR066
+L GND #PWR069
 U 1 1 53A45320
 P 9500 1500
-F 0 "#PWR066" H 9500 1500 30  0001 C CNN
+F 0 "#PWR069" H 9500 1500 30  0001 C CNN
 F 1 "GND" H 9500 1430 30  0001 C CNN
 F 2 "" H 9500 1500 60  0000 C CNN
@@
 $EndComp
 $Comp
-L +3.3V #PWR067
+L +3.3V #PWR070
 U 1 1 53A4534D
 P 9050 1500
-F 0 "#PWR067" H 9050 1460 30  0001 C CNN
+F 0 "#PWR070" H 9050 1460 30  0001 C CNN
 F 1 "+3.3V" H 9050 1610 30  0000 C CNN
 F 2 "" H 9050 1500 60  0000 C CNN
@@
 $EndSheet
 $Comp
-L +5V #PWR068
+L +5V #PWR071
 U 1 1 53A48DD8
 P 3150 10200
-F 0 "#PWR068" H 3150 10290 20  0001 C CNN
+F 0 "#PWR071" H 3150 10290 20  0001 C CNN
 F 1 "+5V" H 3150 10290 30  0000 C CNN
 F 2 "" H 3150 10200 60  0000 C CNN
@@
 SPI/CAN/I2C
 $Comp
-L GND #PWR069
+L GND #PWR072
 U 1 1 53AD2624
 P 1850 1800
-F 0 "#PWR069" H 1850 1800 30  0001 C CNN
+F 0 "#PWR072" H 1850 1800 30  0001 C CNN
 F 1 "GND" H 1850 1730 30  0001 C CNN
 F 2 "" H 1850 1800 60  0000 C CNN
@@
 $EndComp
 $Comp
-L +3.3V #PWR070
+L +3.3V #PWR073
 U 1 1 53C43E5C
 P 2650 2900
-F 0 "#PWR070" H 2650 2860 30  0001 C CNN
+F 0 "#PWR073" H 2650 2860 30  0001 C CNN
 F 1 "+3.3V" H 2650 3010 30  0000 C CNN
 F 2 "" H 2650 2900 60  0000 C CNN
@@
 $EndComp
 $Comp
-L +3.3V #PWR071
+L +3.3V #PWR074
 U 1 1 53C4BB6B
 P 4400 5400
-F 0 "#PWR071" H 4400 5360 30  0001 C CNN
+F 0 "#PWR074" H 4400 5360 30  0001 C CNN
 F 1 "+3.3V" H 4400 5510 30  0000 C CNN
 F 2 "" H 4400 5400 60  0000 C CNN
@@
 $EndComp
 $Comp
-L GND #PWR072
+L GND #PWR075
 U 1 1 53CF920C
 P 4400 7600
-F 0 "#PWR072" H 4400 7600 30  0001 C CNN
+F 0 "#PWR075" H 4400 7600 30  0001 C CNN
 F 1 "GND" H 4400 7530 30  0001 C CNN
 F 2 "" H 4400 7600 60  0000 C CNN
@@
 POW3
 NoConn ~ 12500 9100
-NoConn ~ 8300 7700
 NoConn ~ 15300 7400
 NoConn ~ 15300 7300
 $Comp
-L +3.3V #PWR073
+L +3.3V #PWR076
 U 1 1 53C2CD3E
 P 3600 8450
-F 0 "#PWR073" H 3600 8410 30  0001 C CNN
+F 0 "#PWR076" H 3600 8410 30  0001 C CNN
 F 1 "+3.3V" H 3600 8560 30  0000 C CNN
 F 2 "" H 3600 8450 60  0000 C CNN
@@
 	7700 8050 7600 8050
 $Comp
-L +5V #PWR074
+L +5V #PWR077
 U 1 1 53C7CFF3
 P 7600 8050
-F 0 "#PWR074" H 7600 8140 20  0001 C CNN
+F 0 "#PWR077" H 7600 8140 20  0001 C CNN
 F 1 "+5V" H 7600 8140 30  0000 C CNN
 F 2 "" H 7600 8050 60  0000 C CNN
@@
 	1    0    0    -1
 $EndComp
+Text HLabel 1500 2400 0    60   Input ~ 0
+U36
+Wire Wire Line
+	1500 2400 1800 2400
+Text Label 1800 2400 0    60   ~ 0
+U36_ADC
+Text Label 8300 7700 2    60   ~ 0
+U36_ADC
+Text HLabel 1500 2200 0    60   Input ~ 0
+U10
+Wire Wire Line
+	1500 2200 1800 2200
+Text Label 1800 2200 0    60   ~ 0
+U10_ADC
+Text Label 8300 7600 2    60   ~ 0
+U10_ADC
 $EndSCHEMATC
