File: schematic/ST3232.sch (KiCad schematic (older format))
At the start: 4 parts, among them IC1 ADM233L, J1 DB9, J2 DB9, P17 CONN_2

Commit message: PCB
Other:
- note added: "Main UART (socket)"
- note added: "Reserved UART (plug)"
- note removed: "Main UART"
- note removed: "Reserved UART"
Changed lines of the file:
@@
-EESchema Schematic File Version 2  date Ср 09 июл 2014 18:42:33
+EESchema Schematic File Version 2  date Пт 11 июл 2014 12:31:03
 LIBS:power
 LIBS:device
@@
 Sheet 5 12
 Title "RS-232 level converter"
-Date "9 jul 2014"
+Date "11 jul 2014"
 Rev ""
 Comp "SAO RAS"
@@
 GND
 $Comp
-L GND #PWR085
+L GND #PWR081
 U 1 1 53974EEB
 P 1600 2200
-F 0 "#PWR085" H 1600 2200 30  0001 C CNN
+F 0 "#PWR081" H 1600 2200 30  0001 C CNN
 F 1 "GND" H 1600 2130 30  0001 C CNN
 F 2 "" H 1600 2200 60  0000 C CNN
@@
 	1600 1900 1600 1850
 $Comp
-L GND #PWR086
+L GND #PWR082
 U 1 1 53975227
 P 5250 3400
-F 0 "#PWR086" H 5250 3400 30  0001 C CNN
+F 0 "#PWR082" H 5250 3400 30  0001 C CNN
 F 1 "GND" H 5250 3330 30  0001 C CNN
 F 2 "" H 5250 3400 60  0000 C CNN
@@
 Connection ~ 1750 3950
 $Comp
-L +5V #PWR087
+L +5V #PWR083
 U 1 1 53A48DE6
 P 1600 1850
-F 0 "#PWR087" H 1600 1940 20  0001 C CNN
+F 0 "#PWR083" H 1600 1940 20  0001 C CNN
 F 1 "+5V" H 1600 1940 30  0000 C CNN
 F 2 "" H 1600 1850 60  0000 C CNN
@@
 Connection ~ 2950 2550
 $Comp
-L GND #PWR088
+L GND #PWR084
 U 1 1 53A4A7BE
 P 2850 2600
-F 0 "#PWR088" H 2850 2600 30  0001 C CNN
+F 0 "#PWR084" H 2850 2600 30  0001 C CNN
 F 1 "GND" H 2850 2530 30  0001 C CNN
 F 2 "" H 2850 2600 60  0000 C CNN
@@
 $EndComp
 $Comp
-L +5V #PWR089
+L +5V #PWR085
 U 1 1 53A4A7C4
 P 2950 2250
-F 0 "#PWR089" H 2950 2340 20  0001 C CNN
+F 0 "#PWR085" H 2950 2340 20  0001 C CNN
 F 1 "+5V" H 2950 2340 30  0000 C CNN
 F 2 "" H 2950 2250 60  0000 C CNN
@@
 DB9 pinout:\n1 - Data carrier detect\n2 - Receive data\n3 - Transmit data\n4 - Data terminal ready\n5 - Signal ground\n6 - Data set ready\n7 - Request to send\n8 - Clear to send\n9 - Ring indicator
 Text Notes 5300 2250 0    60   ~ 0
-Main UART
+Main UART (socket)
 NoConn ~ 5250 3200
 NoConn ~ 5250 2800
@@
 NoConn ~ 5250 2500
 $Comp
-L GND #PWR090
+L GND #PWR086
 U 1 1 53AB443D
 P 5250 4800
-F 0 "#PWR090" H 5250 4800 30  0001 C CNN
+F 0 "#PWR086" H 5250 4800 30  0001 C CNN
 F 1 "GND" H 5250 4730 30  0001 C CNN
 F 2 "" H 5250 4800 60  0000 C CNN
@@
 NoConn ~ 5250 4000
 Text Notes 5300 3650 0    60   ~ 0
-Reserved UART
+Reserved UART (plug)
 NoConn ~ 5250 4600
 NoConn ~ 5250 4200

Commit message: last?
Parts:
- removed P17: CONN_2, SIL-2, symbol CONN_2
- renumbered IC1 to DD1, J2 to XP6, J1 to XS1
Other:
- note removed: "CMOS/TTL inout"
Changed lines of the file:
@@
-EESchema Schematic File Version 2  date Пт 11 июл 2014 12:31:03
+EESchema Schematic File Version 2  date Пт 18 июл 2014 12:36:52
 LIBS:power
 LIBS:device
@@
 Sheet 5 12
 Title "RS-232 level converter"
-Date "11 jul 2014"
+Date "18 jul 2014"
 Rev ""
 Comp "SAO RAS"
@@
 GND
 $Comp
-L GND #PWR081
+L GND #PWR079
 U 1 1 53974EEB
 P 1600 2200
-F 0 "#PWR081" H 1600 2200 30  0001 C CNN
+F 0 "#PWR079" H 1600 2200 30  0001 C CNN
 F 1 "GND" H 1600 2130 30  0001 C CNN
 F 2 "" H 1600 2200 60  0000 C CNN
@@
 	1600 1900 1600 1850
 $Comp
-L GND #PWR082
+L GND #PWR080
 U 1 1 53975227
 P 5250 3400
-F 0 "#PWR082" H 5250 3400 30  0001 C CNN
+F 0 "#PWR080" H 5250 3400 30  0001 C CNN
 F 1 "GND" H 5250 3330 30  0001 C CNN
 F 2 "" H 5250 3400 60  0000 C CNN
@@
 $EndComp
 $Comp
-L DB9 J1
+L DB9 XS1
 U 1 1 53975A15
 P 5700 2900
-F 0 "J1" H 5700 3450 70  0000 C CNN
+F 0 "XS1" H 5700 3450 70  0000 C CNN
 F 1 "DB9" H 5700 2350 70  0000 C CNN
 F 2 "DB9FC" H 5700 2900 60  0001 C CNN
@@
 UART_TX1
 $Comp
-L CONN_2 P17
-U 1 1 53A1F05B
-P 1400 3000
-F 0 "P17" V 1350 3000 40  0000 C CNN
-F 1 "CONN_2" V 1450 3000 40  0000 C CNN
-F 2 "SIL-2" H 1400 3000 60  0001 C CNN
-F 3 "" H 1400 3000 60  0000 C CNN
-	1    1400 3000
-	-1   0    0    1
-$EndComp
-Text Notes 1100 2750 0    60   ~ 0
-CMOS/TTL inout
-Wire Wire Line
-	1750 2900 2000 2900
-Wire Wire Line
-	2000 2900 2000 3650
-Connection ~ 2000 3650
-Wire Wire Line
-	1750 3100 1750 3950
-Connection ~ 1750 3950
-$Comp
-L +5V #PWR083
+L +5V #PWR081
 U 1 1 53A48DE6
 P 1600 1850
-F 0 "#PWR083" H 1600 1940 20  0001 C CNN
+F 0 "#PWR081" H 1600 1940 20  0001 C CNN
 F 1 "+5V" H 1600 1940 30  0000 C CNN
 F 2 "" H 1600 1850 60  0000 C CNN
@@
 $EndComp
 $Comp
-L ADM233L IC1
+L ADM233L DD1
 U 1 1 53A48DFB
 P 3450 2650
-F 0 "IC1" H 3250 3100 60  0000 C CNN
+F 0 "DD1" H 3250 3100 60  0000 C CNN
 F 1 "ADM233L" H 3450 1750 60  0000 C CNN
 F 2 "DIP-20__300" H 3450 2650 60  0001 C CNN
@@
 Connection ~ 2950 2550
 $Comp
-L GND #PWR084
+L GND #PWR082
 U 1 1 53A4A7BE
 P 2850 2600
-F 0 "#PWR084" H 2850 2600 30  0001 C CNN
+F 0 "#PWR082" H 2850 2600 30  0001 C CNN
 F 1 "GND" H 2850 2530 30  0001 C CNN
 F 2 "" H 2850 2600 60  0000 C CNN
@@
 $EndComp
 $Comp
-L +5V #PWR085
+L +5V #PWR083
 U 1 1 53A4A7C4
 P 2950 2250
-F 0 "#PWR085" H 2950 2340 20  0001 C CNN
+F 0 "#PWR083" H 2950 2340 20  0001 C CNN
 F 1 "+5V" H 2950 2340 30  0000 C CNN
 F 2 "" H 2950 2250 60  0000 C CNN
@@
 NoConn ~ 5250 2500
 $Comp
-L GND #PWR086
+L GND #PWR084
 U 1 1 53AB443D
 P 5250 4800
-F 0 "#PWR086" H 5250 4800 30  0001 C CNN
+F 0 "#PWR084" H 5250 4800 30  0001 C CNN
 F 1 "GND" H 5250 4730 30  0001 C CNN
 F 2 "" H 5250 4800 60  0000 C CNN
@@
 $EndComp
 $Comp
-L DB9 J2
+L DB9 XP6
 U 1 1 53AB4443
 P 5700 4300
-F 0 "J2" H 5700 4850 70  0000 C CNN
+F 0 "XP6" H 5700 4850 70  0000 C CNN
 F 1 "DB9" H 5700 3750 70  0000 C CNN
 F 2 "DB9FC" H 5700 4300 60  0001 C CNN

Commit message: modified schematics
Parts:
- XP6: value DB9 -> DB9-M; footprint DB9FC -> DB9-M
- XS1: value DB9 -> DB9-F; footprint DB9FC -> DB9-F
Connections:
- net at DD1.18 (T2_O): now also XP6.3; no longer XP6.2
- net at DD1.19 (R2_I): now also XP6.2; no longer XP6.3
Other:
- note added: "Main UART (female)\ncomputer -> MCU"
- note added: "Slave UART (male)\nMCU -> slaves"
- note removed: "Main UART (socket)"
- note removed: "Reserved UART (plug)"
Changed lines of the file:
@@
-EESchema Schematic File Version 2  date Вт 07 окт 2014 17:18:47
+EESchema Schematic File Version 2  date Вс 30 ноя 2014 15:36:58
 LIBS:power
 LIBS:device
@@
 Sheet 5 12
 Title "RS-232 level converter"
-Date "7 oct 2014"
+Date "30 nov 2014"
 Rev ""
 Comp "SAO RAS"
@@
 GND
 $Comp
-L GND #PWR079
+L GND #PWR083
 U 1 1 53974EEB
 P 1600 2200
-F 0 "#PWR079" H 1600 2200 30  0001 C CNN
+F 0 "#PWR083" H 1600 2200 30  0001 C CNN
 F 1 "GND" H 1600 2130 30  0001 C CNN
 F 2 "" H 1600 2200 60  0000 C CNN
@@
 	1600 1900 1600 1850
 $Comp
-L GND #PWR080
+L GND #PWR084
 U 1 1 53975227
 P 5250 3400
-F 0 "#PWR080" H 5250 3400 30  0001 C CNN
+F 0 "#PWR084" H 5250 3400 30  0001 C CNN
 F 1 "GND" H 5250 3330 30  0001 C CNN
 F 2 "" H 5250 3400 60  0000 C CNN
@@
 P 5700 2900
 F 0 "XS1" H 5700 3450 70  0000 C CNN
-F 1 "DB9" H 5700 2350 70  0000 C CNN
-F 2 "DB9FC" H 5700 2900 60  0001 C CNN
+F 1 "DB9-F" H 5700 2350 70  0000 C CNN
+F 2 "DB9-F" H 5700 2900 60  0001 C CNN
 F 3 "" H 5700 2900 60  0000 C CNN
 	1    5700 2900
@@
 UART_TX1
 $Comp
-L +5V #PWR081
+L +5V #PWR085
 U 1 1 53A48DE6
 P 1600 1850
-F 0 "#PWR081" H 1600 1940 20  0001 C CNN
+F 0 "#PWR085" H 1600 1940 20  0001 C CNN
 F 1 "+5V" H 1600 1940 30  0000 C CNN
 F 2 "" H 1600 1850 60  0000 C CNN
@@
 Connection ~ 2950 2550
 $Comp
-L GND #PWR082
+L GND #PWR086
 U 1 1 53A4A7BE
 P 2850 2600
-F 0 "#PWR082" H 2850 2600 30  0001 C CNN
+F 0 "#PWR086" H 2850 2600 30  0001 C CNN
 F 1 "GND" H 2850 2530 30  0001 C CNN
 F 2 "" H 2850 2600 60  0000 C CNN
@@
 $EndComp
 $Comp
-L +5V #PWR083
+L +5V #PWR087
 U 1 1 53A4A7C4
 P 2950 2250
-F 0 "#PWR083" H 2950 2340 20  0001 C CNN
+F 0 "#PWR087" H 2950 2340 20  0001 C CNN
 F 1 "+5V" H 2950 2340 30  0000 C CNN
 F 2 "" H 2950 2250 60  0000 C CNN
@@
 Text Notes 6700 2300 0    100  ~ 0
 DB9 pinout:\n1 - Data carrier detect\n2 - Receive data\n3 - Transmit data\n4 - Data terminal ready\n5 - Signal ground\n6 - Data set ready\n7 - Request to send\n8 - Clear to send\n9 - Ring indicator
-Text Notes 5300 2250 0    60   ~ 0
-Main UART (socket)
+Text Notes 5200 2150 0    60   ~ 0
+Main UART (female)\ncomputer -> MCU
 NoConn ~ 5250 3200
 NoConn ~ 5250 2800
@@
 NoConn ~ 5250 2500
 $Comp
-L GND #PWR084
+L GND #PWR088
 U 1 1 53AB443D
 P 5250 4800
-F 0 "#PWR084" H 5250 4800 30  0001 C CNN
+F 0 "#PWR088" H 5250 4800 30  0001 C CNN
 F 1 "GND" H 5250 4730 30  0001 C CNN
 F 2 "" H 5250 4800 60  0000 C CNN
@@
 P 5700 4300
 F 0 "XP6" H 5700 4850 70  0000 C CNN
-F 1 "DB9" H 5700 3750 70  0000 C CNN
-F 2 "DB9FC" H 5700 4300 60  0001 C CNN
+F 1 "DB9-M" H 5700 3750 70  0000 C CNN
+F 2 "DB9-M" H 5700 4300 60  0001 C CNN
 F 3 "" H 5700 4300 60  0000 C CNN
 	1    5700 4300
@@
 $EndComp
 NoConn ~ 5250 4000
-Text Notes 5300 3650 0    60   ~ 0
-Reserved UART (plug)
+Text Notes 5300 5050 0    60   ~ 0
+Slave UART (male)\nMCU -> slaves
 NoConn ~ 5250 4600
 NoConn ~ 5250 4200
@@
 	3950 2800 4550 2800
 Wire Wire Line
-	4550 2800 4550 4300
-Wire Wire Line
-	4550 4300 5250 4300
-Wire Wire Line
-	5250 4100 4750 4100
-Wire Wire Line
-	4750 4100 4750 2600
+	4750 2600 4750 4300
 Wire Wire Line
 	4750 2600 3950 2600
+Wire Wire Line
+	4750 4300 5250 4300
+Wire Wire Line
+	4550 4100 5250 4100
+Wire Wire Line
+	4550 2800 4550 4100
 $EndSCHEMATC
