File: schematic/Shutter_MOSFET.sch (KiCad schematic (older format))
At the start: 3 parts, among them U2 TLE5205

Commit message: PCB
Parts:
- R25: value 1.2k (II) -> 300 (II)
Changed lines of the file:
@@
-EESchema Schematic File Version 2  date Ср 09 июл 2014 18:42:33
+EESchema Schematic File Version 2  date Пт 11 июл 2014 12:31:03
 LIBS:power
 LIBS:device
@@
 Sheet 12 12
 Title "Power load module"
-Date "9 jul 2014"
+Date "11 jul 2014"
 Rev ""
 Comp "SAO RAS"
@@
 AR Path="/53AA0E2D/53BC59AD" Ref="#PWRp0132"  Part="1"
 AR Path="/53AA0E2C/53BC59AD" Ref="#PWRp0135"  Part="1"
-AR Path="/53AE6F08/53BC59AD" Ref="#PWRp0135"  Part="1"
-F 0 "#PWRp0135" H 2450 2100 30  0001 C CNN
+AR Path="/53AE6F08/53BC59AD" Ref="#PWRp0131"  Part="1"
+F 0 "#PWRp0131" H 2450 2100 30  0001 C CNN
 F 1 "GND" H 2450 2030 30  0001 C CNN
 F 2 "" H 2450 2100 60  0000 C CNN
@@
 	4600 5200 2350 5200
 $Comp
-L GND #PWRp0136
+L GND #PWRp0132
 U 1 1 53C0B3EC
 P 3500 4350
-F 0 "#PWRp0136" H 3500 4350 30  0001 C CNN
+F 0 "#PWRp0132" H 3500 4350 30  0001 C CNN
 F 1 "GND" H 3500 4280 30  0001 C CNN
 F 2 "" H 3500 4350 60  0000 C CNN
@@
 +36V
 $Comp
-L GND #PWRp0137
+L GND #PWRp0133
 U 1 1 53C0BE69
 P 3900 2500
-F 0 "#PWRp0137" H 3900 2500 30  0001 C CNN
+F 0 "#PWRp0133" H 3900 2500 30  0001 C CNN
 F 1 "GND" H 3900 2430 30  0001 C CNN
 F 2 "" H 3900 2500 60  0000 C CNN
@@
 P 3000 2400
 F 0 "R25" V 3080 2400 40  0000 C CNN
-F 1 "1.2k (II)" V 3007 2401 40  0000 C CNN
+F 1 "300 (II)" V 3007 2401 40  0000 C CNN
 F 2 "R7" V 2930 2400 30  0001 C CNN
 F 3 "~" H 3000 2400 30  0000 C CNN
@@
 	4600 3800 4600 5200
 $Comp
-L PWR_FLAG #FLG0138
+L PWR_FLAG #FLG0134
 U 1 1 53CB51C4
 P 3350 2400
-F 0 "#FLG0138" H 3350 2495 30  0001 C CNN
+F 0 "#FLG0134" H 3350 2495 30  0001 C CNN
 F 1 "PWR_FLAG" H 3350 2580 30  0000 C CNN
 F 2 "" H 3350 2400 60  0000 C CNN

Commit message: last?
Parts:
- renumbered U2 to DA2
Changed lines of the file:
@@
-EESchema Schematic File Version 2  date Пт 11 июл 2014 12:31:03
+EESchema Schematic File Version 2  date Пт 18 июл 2014 12:36:52
 LIBS:power
 LIBS:device
@@
 Sheet 12 12
 Title "Power load module"
-Date "11 jul 2014"
+Date "18 jul 2014"
 Rev ""
 Comp "SAO RAS"
@@
 AR Path="/53AA0E2D/53BC59AD" Ref="#PWRp0132"  Part="1"
 AR Path="/53AA0E2C/53BC59AD" Ref="#PWRp0135"  Part="1"
-AR Path="/53AE6F08/53BC59AD" Ref="#PWRp0131"  Part="1"
-F 0 "#PWRp0131" H 2450 2100 30  0001 C CNN
+AR Path="/53AE6F08/53BC59AD" Ref="#PWRp0129"  Part="1"
+F 0 "#PWRp0129" H 2450 2100 30  0001 C CNN
 F 1 "GND" H 2450 2030 30  0001 C CNN
 F 2 "" H 2450 2100 60  0000 C CNN
@@
 	2450 2000 2450 2100
 $Comp
-L TLE5205 U2
+L TLE5205 DA2
 U 1 1 53C09F3E
 P 3500 3650
-F 0 "U2" H 3650 4050 60  0000 C CNN
+F 0 "DA2" H 3650 4050 60  0000 C CNN
 F 1 "TLE5205" H 3500 3650 60  0000 C CNN
 F 2 "TO220-7-12" H 3500 3650 60  0001 C CNN
@@
 	4600 5200 2350 5200
 $Comp
-L GND #PWRp0132
+L GND #PWRp0130
 U 1 1 53C0B3EC
 P 3500 4350
-F 0 "#PWRp0132" H 3500 4350 30  0001 C CNN
+F 0 "#PWRp0130" H 3500 4350 30  0001 C CNN
 F 1 "GND" H 3500 4280 30  0001 C CNN
 F 2 "" H 3500 4350 60  0000 C CNN
@@
 +36V
 $Comp
-L GND #PWRp0133
+L GND #PWRp0131
 U 1 1 53C0BE69
 P 3900 2500
-F 0 "#PWRp0133" H 3900 2500 30  0001 C CNN
+F 0 "#PWRp0131" H 3900 2500 30  0001 C CNN
 F 1 "GND" H 3900 2430 30  0001 C CNN
 F 2 "" H 3900 2500 60  0000 C CNN
@@
 	4600 3800 4600 5200
 $Comp
-L PWR_FLAG #FLG0134
+L PWR_FLAG #FLG0132
 U 1 1 53CB51C4
 P 3350 2400
-F 0 "#FLG0134" H 3350 2495 30  0001 C CNN
+F 0 "#FLG0132" H 3350 2495 30  0001 C CNN
 F 1 "PWR_FLAG" H 3350 2580 30  0000 C CNN
 F 2 "" H 3350 2400 60  0000 C CNN

Commit message: modified schematics
Parts:
- added R41: 56k, SM0603, symbol R0603
- added R42: 4.7k, SM0603, symbol R0603
Connections:
- net GND: now also R42.2
- net at C4.1, DA2.6 (Vs), R25.2: now also R41.1
- new net Sense: R41.2, R42.1
Other:
- note added: "2W!"
- note removed: "2Вт!"
Changed lines of the file:
@@
-EESchema Schematic File Version 2  date Вт 07 окт 2014 17:18:47
+EESchema Schematic File Version 2  date Вс 30 ноя 2014 15:36:58
 LIBS:power
 LIBS:device
@@
 Sheet 12 12
 Title "Power load module"
-Date "7 oct 2014"
+Date "30 nov 2014"
 Rev ""
 Comp "SAO RAS"
@@
 AR Path="/53AA0E2D/53BC59AD" Ref="#PWRp0132"  Part="1"
 AR Path="/53AA0E2C/53BC59AD" Ref="#PWRp0135"  Part="1"
-AR Path="/53AE6F08/53BC59AD" Ref="#PWRp0129"  Part="1"
-F 0 "#PWRp0129" H 2450 2100 30  0001 C CNN
+AR Path="/53AE6F08/53BC59AD" Ref="#PWRp0133"  Part="1"
+F 0 "#PWRp0133" H 2450 2100 30  0001 C CNN
 F 1 "GND" H 2450 2030 30  0001 C CNN
 F 2 "" H 2450 2100 60  0000 C CNN
@@
 	2350 2000 2450 2000
 Wire Wire Line
-	2450 2000 2450 2100
+	2450 1950 2450 2100
 $Comp
 L TLE5205 DA2
@@
 	4600 5200 2350 5200
 $Comp
-L GND #PWRp0130
+L GND #PWRp0134
 U 1 1 53C0B3EC
 P 3500 4350
-F 0 "#PWRp0130" H 3500 4350 30  0001 C CNN
+F 0 "#PWRp0134" H 3500 4350 30  0001 C CNN
 F 1 "GND" H 3500 4280 30  0001 C CNN
 F 2 "" H 3500 4350 60  0000 C CNN
@@
 +36V
 $Comp
-L GND #PWRp0131
+L GND #PWRp0135
 U 1 1 53C0BE69
 P 3900 2500
-F 0 "#PWRp0131" H 3900 2500 30  0001 C CNN
+F 0 "#PWRp0135" H 3900 2500 30  0001 C CNN
 F 1 "GND" H 3900 2430 30  0001 C CNN
 F 2 "" H 3900 2500 60  0000 C CNN
@@
 $EndComp
 Text Notes 2900 2550 0    60   ~ 0
-2Вт!
+2W!
 Wire Wire Line
 	2350 2400 2750 2400
@@
 	3250 2400 3500 2400
 Wire Wire Line
-	3500 2400 3500 3050
+	3500 850  3500 3050
 Connection ~ 3500 2400
 $Comp
@@
 	4600 3800 4600 5200
 $Comp
-L PWR_FLAG #FLG0132
+L PWR_FLAG #FLG0136
 U 1 1 53CB51C4
 P 3350 2400
-F 0 "#FLG0132" H 3350 2495 30  0001 C CNN
+F 0 "#FLG0136" H 3350 2495 30  0001 C CNN
 F 1 "PWR_FLAG" H 3350 2580 30  0000 C CNN
 F 2 "" H 3350 2400 60  0000 C CNN
@@
 $EndComp
 Connection ~ 3350 2400
+$Comp
+L R0603 R42
+U 1 1 5465870A
+P 2450 1700
+F 0 "R42" V 2530 1700 40  0000 C CNN
+F 1 "4.7k" V 2457 1701 40  0000 C CNN
+F 2 "SM0603" V 2380 1700 30  0001 C CNN
+F 3 "~" H 2450 1700 30  0000 C CNN
+	1    2450 1700
+	1    0    0    -1
+$EndComp
+$Comp
+L R0603 R41
+U 1 1 54658717
+P 2450 1100
+F 0 "R41" V 2530 1100 40  0000 C CNN
+F 1 "56k" V 2457 1101 40  0000 C CNN
+F 2 "SM0603" V 2380 1100 30  0001 C CNN
+F 3 "~" H 2450 1100 30  0000 C CNN
+	1    2450 1100
+	1    0    0    -1
+$EndComp
+Wire Wire Line
+	2450 850  3500 850
+Wire Wire Line
+	2450 1350 2450 1450
+Wire Wire Line
+	2350 1400 2450 1400
+Connection ~ 2450 1400
+Text HLabel 2350 1400 0    60   Output ~ 0
+Sense
+Connection ~ 2450 2000
 $EndSCHEMATC
