File: schematic/motors.sch (KiCad schematic (older format))
At the start: 10 parts, among them IC2.1 L6208N

Commit message: PCB
Changed lines of the file:
@@
-EESchema Schematic File Version 2  date Ср 09 июл 2014 18:42:33
+EESchema Schematic File Version 2  date Пт 11 июл 2014 12:31:03
 LIBS:power
 LIBS:device
@@
 Sheet 2 12
 Title "Stepper motor module"
-Date "9 jul 2014"
+Date "11 jul 2014"
 Rev ""
 Comp "SAO RAS"
@@
 AR Path="/53A910BA/50CECA5D" Ref="C3.4"  Part="1"
 AR Path="/53A910B9/50CECA5D" Ref="C3.5"  Part="1"
-F 0 "C3.1" H 5550 3350 50  0000 L CNN
+F 0 "C3.5" H 5550 3350 50  0000 L CNN
 F 1 "1n" H 5550 3150 50  0000 L CNN
 F 2 "SM0805" H 5500 3250 60  0001 C CNN
@@
 AR Path="/53A910BA/50CECA5C" Ref="R6.4"  Part="1"
 AR Path="/53A910B9/50CECA5C" Ref="R6.5"  Part="1"
-F 0 "R6.1" V 5580 3000 50  0000 C CNN
+F 0 "R6.5" V 5580 3000 50  0000 C CNN
 F 1 "51k" V 5500 3000 50  0000 C CNN
 F 2 "SM0603" H 5500 3000 60  0001 C CNN
@@
 P 5250 3300
 AR Path="/53A910B8/50CECA5B" Ref="#PWR033"  Part="1"
-AR Path="/53A910B7/50CECA5B" Ref="#PWR091"  Part="1"
-AR Path="/5391724D/50CECA5B" Ref="#PWR0101"  Part="1"
-AR Path="/53A910BA/50CECA5B" Ref="#PWR0111"  Part="1"
-AR Path="/53A910B9/50CECA5B" Ref="#PWR0121"  Part="1"
-F 0 "#PWR0121" H 5250 3300 30  0001 C CNN
+AR Path="/53A910B7/50CECA5B" Ref="#PWR087"  Part="1"
+AR Path="/5391724D/50CECA5B" Ref="#PWR097"  Part="1"
+AR Path="/53A910BA/50CECA5B" Ref="#PWR0107"  Part="1"
+AR Path="/53A910B9/50CECA5B" Ref="#PWR0117"  Part="1"
+F 0 "#PWR0117" H 5250 3300 30  0001 C CNN
 F 1 "GND" H 5250 3230 30  0001 C CNN
 F 2 "" H 5250 3300 60  0001 C CNN
@@
 P 3850 2700
 AR Path="/53A910B8/50CEC8BA" Ref="#PWR034"  Part="1"
-AR Path="/53A910B7/50CEC8BA" Ref="#PWR092"  Part="1"
-AR Path="/5391724D/50CEC8BA" Ref="#PWR0102"  Part="1"
-AR Path="/53A910BA/50CEC8BA" Ref="#PWR0112"  Part="1"
-AR Path="/53A910B9/50CEC8BA" Ref="#PWR0122"  Part="1"
-F 0 "#PWR0122" H 3850 2700 30  0001 C CNN
+AR Path="/53A910B7/50CEC8BA" Ref="#PWR088"  Part="1"
+AR Path="/5391724D/50CEC8BA" Ref="#PWR098"  Part="1"
+AR Path="/53A910BA/50CEC8BA" Ref="#PWR0108"  Part="1"
+AR Path="/53A910B9/50CEC8BA" Ref="#PWR0118"  Part="1"
+F 0 "#PWR0118" H 3850 2700 30  0001 C CNN
 F 1 "GND" H 3850 2630 30  0001 C CNN
 F 2 "" H 3850 2700 60  0001 C CNN
@@
 P 5250 2800
 AR Path="/53A910B8/50CEC869" Ref="#PWR035"  Part="1"
-AR Path="/53A910B7/50CEC869" Ref="#PWR093"  Part="1"
-AR Path="/5391724D/50CEC869" Ref="#PWR0103"  Part="1"
-AR Path="/53A910BA/50CEC869" Ref="#PWR0113"  Part="1"
-AR Path="/53A910B9/50CEC869" Ref="#PWR0123"  Part="1"
-F 0 "#PWR0123" H 5250 2800 30  0001 C CNN
+AR Path="/53A910B7/50CEC869" Ref="#PWR089"  Part="1"
+AR Path="/5391724D/50CEC869" Ref="#PWR099"  Part="1"
+AR Path="/53A910BA/50CEC869" Ref="#PWR0109"  Part="1"
+AR Path="/53A910B9/50CEC869" Ref="#PWR0119"  Part="1"
+F 0 "#PWR0119" H 5250 2800 30  0001 C CNN
 F 1 "GND" H 5250 2730 30  0001 C CNN
 F 2 "" H 5250 2800 60  0001 C CNN
@@
 AR Path="/53A910BA/50CEC791" Ref="R5.4"  Part="1"
 AR Path="/53A910B9/50CEC791" Ref="R5.5"  Part="1"
-F 0 "R5.1" V 5580 2500 50  0000 C CNN
+F 0 "R5.5" V 5580 2500 50  0000 C CNN
 F 1 "51k" V 5500 2500 50  0000 C CNN
 F 2 "SM0603" H 5500 2500 60  0001 C CNN
@@
 AR Path="/53A910BA/50CEC790" Ref="C2.4"  Part="1"
 AR Path="/53A910B9/50CEC790" Ref="C2.5"  Part="1"
-F 0 "C2.1" H 5550 2850 50  0000 L CNN
+F 0 "C2.5" H 5550 2850 50  0000 L CNN
 F 1 "1n" H 5550 2650 50  0000 L CNN
 F 2 "SM0805" H 5500 2750 60  0001 C CNN
@@
 AR Path="/53A910BA/50CEB99A" Ref="R2.4"  Part="1"
 AR Path="/53A910B9/50CEB99A" Ref="R2.5"  Part="1"
-F 0 "R2.1" V 4280 2650 50  0000 C CNN
+F 0 "R2.5" V 4280 2650 50  0000 C CNN
 F 1 "0.33" V 4200 2650 50  0000 C CNN
 F 2 "SM1210" H 4200 2650 60  0001 C CNN
@@
 AR Path="/53A910BA/50CEB97A" Ref="R1.4"  Part="1"
 AR Path="/53A910B9/50CEB97A" Ref="R1.5"  Part="1"
-F 0 "R1.1" V 4280 2450 50  0000 C CNN
+F 0 "R1.5" V 4280 2450 50  0000 C CNN
 F 1 "0.33" V 4200 2450 50  0000 C CNN
 F 2 "SM1210" H 4200 2450 60  0001 C CNN
@@
 P 3300 3650
 AR Path="/53A910B8/50AF2385" Ref="#PWR036"  Part="1"
-AR Path="/53A910B7/50AF2385" Ref="#PWR094"  Part="1"
-AR Path="/5391724D/50AF2385" Ref="#PWR0104"  Part="1"
-AR Path="/53A910BA/50AF2385" Ref="#PWR0114"  Part="1"
-AR Path="/53A910B9/50AF2385" Ref="#PWR0124"  Part="1"
-F 0 "#PWR0124" H 3300 3740 20  0001 C CNN
+AR Path="/53A910B7/50AF2385" Ref="#PWR090"  Part="1"
+AR Path="/5391724D/50AF2385" Ref="#PWR0100"  Part="1"
+AR Path="/53A910BA/50AF2385" Ref="#PWR0110"  Part="1"
+AR Path="/53A910B9/50AF2385" Ref="#PWR0120"  Part="1"
+F 0 "#PWR0120" H 3300 3740 20  0001 C CNN
 F 1 "+5V" H 3300 3740 30  0000 C CNN
 F 2 "" H 3300 3650 60  0001 C CNN
@@
 P 4050 4800
 AR Path="/53A910B8/50AF2313" Ref="#PWR037"  Part="1"
-AR Path="/53A910B7/50AF2313" Ref="#PWR095"  Part="1"
-AR Path="/5391724D/50AF2313" Ref="#PWR0105"  Part="1"
-AR Path="/53A910BA/50AF2313" Ref="#PWR0115"  Part="1"
-AR Path="/53A910B9/50AF2313" Ref="#PWR0125"  Part="1"
-F 0 "#PWR0125" H 4050 4800 30  0001 C CNN
+AR Path="/53A910B7/50AF2313" Ref="#PWR091"  Part="1"
+AR Path="/5391724D/50AF2313" Ref="#PWR0101"  Part="1"
+AR Path="/53A910BA/50AF2313" Ref="#PWR0111"  Part="1"
+AR Path="/53A910B9/50AF2313" Ref="#PWR0121"  Part="1"
+F 0 "#PWR0121" H 4050 4800 30  0001 C CNN
 F 1 "GND" H 4050 4730 30  0001 C CNN
 F 2 "" H 4050 4800 60  0001 C CNN
@@
 AR Path="/53A910BA/50AF1E60" Ref="C1.4"  Part="1"
 AR Path="/53A910B9/50AF1E60" Ref="C1.5"  Part="1"
-F 0 "C1.1" H 5100 5100 50  0000 L CNN
+F 0 "C1.5" H 5100 5100 50  0000 L CNN
 F 1 "68n" H 5100 4900 50  0000 L CNN
 F 2 "SM0805" H 5050 5000 60  0001 C CNN
@@
 P 4850 5450
 AR Path="/53A910B8/50AF1E09" Ref="#PWR038"  Part="1"
-AR Path="/53A910B7/50AF1E09" Ref="#PWR096"  Part="1"
-AR Path="/5391724D/50AF1E09" Ref="#PWR0106"  Part="1"
-AR Path="/53A910BA/50AF1E09" Ref="#PWR0116"  Part="1"
-AR Path="/53A910B9/50AF1E09" Ref="#PWR0126"  Part="1"
-F 0 "#PWR0126" H 4850 5450 30  0001 C CNN
+AR Path="/53A910B7/50AF1E09" Ref="#PWR092"  Part="1"
+AR Path="/5391724D/50AF1E09" Ref="#PWR0102"  Part="1"
+AR Path="/53A910BA/50AF1E09" Ref="#PWR0112"  Part="1"
+AR Path="/53A910B9/50AF1E09" Ref="#PWR0122"  Part="1"
+F 0 "#PWR0122" H 4850 5450 30  0001 C CNN
 F 1 "GND" H 4850 5380 30  0001 C CNN
 F 2 "" H 4850 5450 60  0001 C CNN
@@
 P 4400 5400
 AR Path="/53A910B8/50AF1DE3" Ref="#PWR039"  Part="1"
-AR Path="/53A910B7/50AF1DE3" Ref="#PWR097"  Part="1"
-AR Path="/5391724D/50AF1DE3" Ref="#PWR0107"  Part="1"
-AR Path="/53A910BA/50AF1DE3" Ref="#PWR0117"  Part="1"
-AR Path="/53A910B9/50AF1DE3" Ref="#PWR0127"  Part="1"
-F 0 "#PWR0127" H 4400 5490 20  0001 C CNN
+AR Path="/53A910B7/50AF1DE3" Ref="#PWR093"  Part="1"
+AR Path="/5391724D/50AF1DE3" Ref="#PWR0103"  Part="1"
+AR Path="/53A910BA/50AF1DE3" Ref="#PWR0113"  Part="1"
+AR Path="/53A910B9/50AF1DE3" Ref="#PWR0123"  Part="1"
+F 0 "#PWR0123" H 4400 5490 20  0001 C CNN
 F 1 "+5V" H 4400 5490 30  0000 C CNN
 F 2 "" H 4400 5400 60  0001 C CNN
@@
 AR Path="/53A910BA/50AF1C25" Ref="R3.4"  Part="1"
 AR Path="/53A910B9/50AF1C25" Ref="R3.5"  Part="1"
-F 0 "R3.1" V 4480 5050 50  0000 C CNN
+F 0 "R3.5" V 4480 5050 50  0000 C CNN
 F 1 "22k" V 4400 5050 50  0000 C CNN
 F 2 "SM0603" H 4400 5050 60  0001 C CNN
@@
 AR Path="/53A910BA/50AE2A4D" Ref="IC2.4"  Part="1"
 AR Path="/53A910B9/50AE2A4D" Ref="IC2.5"  Part="1"
-F 0 "IC2.1" H 3800 4600 50  0000 L BNN
+F 0 "IC2.5" H 3800 4600 50  0000 L BNN
 F 1 "L6208N" H 4300 2850 50  0000 L BNN
 F 2 "DIP-24__300_ELL" H 4300 3900 50  0001 C CNN
@@
 P 3650 3750
 AR Path="/53A910B8/534B86E7" Ref="#PWR040"  Part="1"
-AR Path="/53A910B7/534B86E7" Ref="#PWR098"  Part="1"
-AR Path="/5391724D/534B86E7" Ref="#PWR0108"  Part="1"
-AR Path="/53A910BA/534B86E7" Ref="#PWR0118"  Part="1"
-AR Path="/53A910B9/534B86E7" Ref="#PWR0128"  Part="1"
-F 0 "#PWR0128" H 3650 3750 30  0001 C CNN
+AR Path="/53A910B7/534B86E7" Ref="#PWR094"  Part="1"
+AR Path="/5391724D/534B86E7" Ref="#PWR0104"  Part="1"
+AR Path="/53A910BA/534B86E7" Ref="#PWR0114"  Part="1"
+AR Path="/53A910B9/534B86E7" Ref="#PWR0124"  Part="1"
+F 0 "#PWR0124" H 3650 3750 30  0001 C CNN
 F 1 "GND" H 3650 3680 30  0001 C CNN
 F 2 "" H 3650 3750 60  0000 C CNN
@@
 AR Path="/53A910BA/534BB108" Ref="R4.4"  Part="1"
 AR Path="/53A910B9/534BB108" Ref="R4.5"  Part="1"
-F 0 "R4.1" V 4780 5050 40  0000 C CNN
+F 0 "R4.5" V 4780 5050 40  0000 C CNN
 F 1 "1.8k" V 4707 5051 40  0000 C CNN
 F 2 "SM0603" V 4630 5050 30  0001 C CNN
@@
 P 2800 2700
 AR Path="/53A910B8/5396FC14" Ref="#PWR041"  Part="1"
-AR Path="/53A910B7/5396FC14" Ref="#PWR099"  Part="1"
-AR Path="/5391724D/5396FC14" Ref="#PWR0109"  Part="1"
-AR Path="/53A910BA/5396FC14" Ref="#PWR0119"  Part="1"
-AR Path="/53A910B9/5396FC14" Ref="#PWR0129"  Part="1"
-F 0 "#PWR0129" H 2800 2790 20  0001 C CNN
+AR Path="/53A910B7/5396FC14" Ref="#PWR095"  Part="1"
+AR Path="/5391724D/5396FC14" Ref="#PWR0105"  Part="1"
+AR Path="/53A910BA/5396FC14" Ref="#PWR0115"  Part="1"
+AR Path="/53A910B9/5396FC14" Ref="#PWR0125"  Part="1"
+F 0 "#PWR0125" H 2800 2790 20  0001 C CNN
 F 1 "+5V" H 2800 2790 30  0000 C CNN
 F 2 "" H 2800 2700 60  0001 C CNN
@@
 P 2700 3150
 AR Path="/53A910B8/53A16DEA" Ref="#PWR042"  Part="1"
-AR Path="/53A910B7/53A16DEA" Ref="#PWR0100"  Part="1"
-AR Path="/5391724D/53A16DEA" Ref="#PWR0110"  Part="1"
-AR Path="/53A910BA/53A16DEA" Ref="#PWR0120"  Part="1"
-AR Path="/53A910B9/53A16DEA" Ref="#PWR0130"  Part="1"
-F 0 "#PWR0130" H 2700 3150 30  0001 C CNN
+AR Path="/53A910B7/53A16DEA" Ref="#PWR096"  Part="1"
+AR Path="/5391724D/53A16DEA" Ref="#PWR0106"  Part="1"
+AR Path="/53A910BA/53A16DEA" Ref="#PWR0116"  Part="1"
+AR Path="/53A910B9/53A16DEA" Ref="#PWR0126"  Part="1"
+F 0 "#PWR0126" H 2700 3150 30  0001 C CNN
 F 1 "GND" H 2700 3080 30  0001 C CNN
 F 2 "" H 2700 3150 60  0001 C CNN

Commit message: last?
Parts:
- renumbered IC2.1 to DD2.1

Commit message: modified schematics
Parts:
- R1.1, R2.1: footprint SM1210 -> SM2010
