File: schematic/power_MOSFET.sch (KiCad schematic (older format))
At the start: 1 part

Commit message: PCB
Changed lines of the file:
@@
-EESchema Schematic File Version 2  date Ср 09 июл 2014 18:42:33
+EESchema Schematic File Version 2  date Пт 11 июл 2014 12:31:03
 LIBS:power
 LIBS:device
@@
 Sheet 10 12
 Title "Power load module"
-Date "9 jul 2014"
+Date "11 jul 2014"
 Rev ""
 Comp "SAO RAS"
@@
 AR Path="/53C7395A/53AF4F61" Ref="#PWRp0140"  Part="1"
 AR Path="/53C73958/53AF4F61" Ref="#PWRp086"  Part="1"
-AR Path="/53A8FBFD/53AF4F61" Ref="#PWRp0131"  Part="1"
-AR Path="/53AA0E2D/53AF4F61" Ref="#PWRp0133"  Part="1"
+AR Path="/53A8FBFD/53AF4F61" Ref="#PWRp0127"  Part="1"
+AR Path="/53AA0E2D/53AF4F61" Ref="#PWRp0129"  Part="1"
 AR Path="/53AA0E2C/53AF4F61" Ref="#PWRp0135"  Part="1"
-F 0 "#PWRp0133" H 3300 2900 30  0001 C CNN
+F 0 "#PWRp0129" H 3300 2900 30  0001 C CNN
 F 1 "GND" H 3300 2830 30  0001 C CNN
 F 2 "" H 3300 2900 60  0000 C CNN
@@
 AR Path="/53AA0E2D/53AF4F62" Ref="Qp1.1"  Part="1"
 AR Path="/53AA0E2C/53AF4F62" Ref="Qp1.2"  Part="1"
-F 0 "Qp1.1" H 4970 2790 60  0000 R CNN
+F 0 "Qp1.2" H 4970 2790 60  0000 R CNN
 F 1 "NTE2984" H 5090 2310 60  0000 R CNN
 F 2 "TO220-3-vert" H 5050 2550 60  0001 C CNN
@@
 AR Path="/53C7395A/53AF4F63" Ref="#PWRp0141"  Part="1"
 AR Path="/53C73958/53AF4F63" Ref="#PWRp087"  Part="1"
-AR Path="/53A8FBFD/53AF4F63" Ref="#PWRp0132"  Part="1"
-AR Path="/53AA0E2D/53AF4F63" Ref="#PWRp0134"  Part="1"
+AR Path="/53A8FBFD/53AF4F63" Ref="#PWRp0128"  Part="1"
+AR Path="/53AA0E2D/53AF4F63" Ref="#PWRp0130"  Part="1"
 AR Path="/53AA0E2C/53AF4F63" Ref="#PWRp0136"  Part="1"
-F 0 "#PWRp0134" H 5150 2850 30  0001 C CNN
+F 0 "#PWRp0130" H 5150 2850 30  0001 C CNN
 F 1 "GND" H 5150 2780 30  0001 C CNN
 F 2 "" H 5150 2850 60  0000 C CNN

Commit message: last?
Parts:
- added R40.2: 68, SM1206, symbol R1206
Connections:
- wire segments 6 -> 7
Changed lines of the file:
@@
-EESchema Schematic File Version 2  date Пт 11 июл 2014 12:31:03
+EESchema Schematic File Version 2  date Пт 18 июл 2014 12:36:52
 LIBS:power
 LIBS:device
@@
 $Descr A4 11693 8268
 encoding utf-8
-Sheet 10 12
+Sheet 11 12
 Title "Power load module"
-Date "11 jul 2014"
+Date "18 jul 2014"
 Rev ""
 Comp "SAO RAS"
@@
 AR Path="/53C7395A/53AF4F61" Ref="#PWRp0140"  Part="1"
 AR Path="/53C73958/53AF4F61" Ref="#PWRp086"  Part="1"
-AR Path="/53A8FBFD/53AF4F61" Ref="#PWRp0127"  Part="1"
-AR Path="/53AA0E2D/53AF4F61" Ref="#PWRp0129"  Part="1"
+AR Path="/53A8FBFD/53AF4F61" Ref="#PWRp0125"  Part="1"
+AR Path="/53AA0E2D/53AF4F61" Ref="#PWRp0127"  Part="1"
 AR Path="/53AA0E2C/53AF4F61" Ref="#PWRp0135"  Part="1"
-F 0 "#PWRp0129" H 3300 2900 30  0001 C CNN
+F 0 "#PWRp0127" H 3300 2900 30  0001 C CNN
 F 1 "GND" H 3300 2830 30  0001 C CNN
 F 2 "" H 3300 2900 60  0000 C CNN
@@
 AR Path="/53C7395A/53AF4F62" Ref="Qp1.3"  Part="1"
 AR Path="/53C73958/53AF4F62" Ref="Qp1.1"  Part="1"
-AR Path="/53A8FBFD/53AF4F62" Ref="Qp1.2"  Part="1"
-AR Path="/53AA0E2D/53AF4F62" Ref="Qp1.1"  Part="1"
+AR Path="/53A8FBFD/53AF4F62" Ref="VT2.2"  Part="1"
+AR Path="/53AA0E2D/53AF4F62" Ref="VT2.1"  Part="1"
 AR Path="/53AA0E2C/53AF4F62" Ref="Qp1.2"  Part="1"
-F 0 "Qp1.2" H 4970 2790 60  0000 R CNN
+F 0 "VT2.1" H 4970 2790 60  0000 R CNN
 F 1 "NTE2984" H 5090 2310 60  0000 R CNN
 F 2 "TO220-3-vert" H 5050 2550 60  0001 C CNN
@@
 	1    0    0    -1
 $EndComp
-Wire Wire Line
-	3200 2550 4850 2550
 Wire Wire Line
 	3150 1250 5150 1250
@@
 AR Path="/53C7395A/53AF4F63" Ref="#PWRp0141"  Part="1"
 AR Path="/53C73958/53AF4F63" Ref="#PWRp087"  Part="1"
-AR Path="/53A8FBFD/53AF4F63" Ref="#PWRp0128"  Part="1"
-AR Path="/53AA0E2D/53AF4F63" Ref="#PWRp0130"  Part="1"
+AR Path="/53A8FBFD/53AF4F63" Ref="#PWRp0126"  Part="1"
+AR Path="/53AA0E2D/53AF4F63" Ref="#PWRp0128"  Part="1"
 AR Path="/53AA0E2C/53AF4F63" Ref="#PWRp0136"  Part="1"
-F 0 "#PWRp0130" H 5150 2850 30  0001 C CNN
+F 0 "#PWRp0128" H 5150 2850 30  0001 C CNN
 F 1 "GND" H 5150 2780 30  0001 C CNN
 F 2 "" H 5150 2850 60  0000 C CNN
@@
 Wire Wire Line
 	5150 2850 5150 2750
+$Comp
+L R1206 R40.2
+U 1 1 53C8FF70
+P 4450 2550
+AR Path="/53A8FBFD/53C8FF70" Ref="R40.2"  Part="1"
+AR Path="/53AA0E2D/53C8FF70" Ref="R40.1"  Part="1"
+F 0 "R40.1" V 4530 2550 40  0000 C CNN
+F 1 "68" V 4457 2551 40  0000 C CNN
+F 2 "SM1206" V 4380 2550 30  0001 C CNN
+F 3 "~" H 4450 2550 30  0000 C CNN
+	1    4450 2550
+	0    -1   -1   0
+$EndComp
+Wire Wire Line
+	3200 2550 4200 2550
+Wire Wire Line
+	4700 2550 4850 2550
 $EndSCHEMATC

Commit message: modified schematics
Parts:
- Qp1.1: value NTE2984 -> FQP30N06
Changed lines of the file:
@@
-EESchema Schematic File Version 2  date Вт 07 окт 2014 17:18:47
+EESchema Schematic File Version 2  date Вс 30 ноя 2014 15:36:58
 LIBS:power
 LIBS:device
@@
 Sheet 11 12
 Title "Power load module"
-Date "7 oct 2014"
+Date "30 nov 2014"
 Rev ""
 Comp "SAO RAS"
@@
 AR Path="/53C7395A/53AF4F61" Ref="#PWRp0140"  Part="1"
 AR Path="/53C73958/53AF4F61" Ref="#PWRp086"  Part="1"
-AR Path="/53A8FBFD/53AF4F61" Ref="#PWRp0125"  Part="1"
-AR Path="/53AA0E2D/53AF4F61" Ref="#PWRp0127"  Part="1"
+AR Path="/53A8FBFD/53AF4F61" Ref="#PWRp0129"  Part="1"
+AR Path="/53AA0E2D/53AF4F61" Ref="#PWRp0131"  Part="1"
 AR Path="/53AA0E2C/53AF4F61" Ref="#PWRp0135"  Part="1"
-F 0 "#PWRp0127" H 3300 2900 30  0001 C CNN
+F 0 "#PWRp0131" H 3300 2900 30  0001 C CNN
 F 1 "GND" H 3300 2830 30  0001 C CNN
 F 2 "" H 3300 2900 60  0000 C CNN
@@
 AR Path="/53AA0E2C/53AF4F62" Ref="Qp1.2"  Part="1"
 F 0 "VT2.1" H 4970 2790 60  0000 R CNN
-F 1 "NTE2984" H 5090 2310 60  0000 R CNN
+F 1 "FQP30N06" H 5090 2310 60  0000 R CNN
 F 2 "TO220-3-vert" H 5050 2550 60  0001 C CNN
 F 3 "~" H 5050 2550 60  0000 C CNN
@@
 AR Path="/53C7395A/53AF4F63" Ref="#PWRp0141"  Part="1"
 AR Path="/53C73958/53AF4F63" Ref="#PWRp087"  Part="1"
-AR Path="/53A8FBFD/53AF4F63" Ref="#PWRp0126"  Part="1"
-AR Path="/53AA0E2D/53AF4F63" Ref="#PWRp0128"  Part="1"
+AR Path="/53A8FBFD/53AF4F63" Ref="#PWRp0130"  Part="1"
+AR Path="/53AA0E2D/53AF4F63" Ref="#PWRp0132"  Part="1"
 AR Path="/53AA0E2C/53AF4F63" Ref="#PWRp0136"  Part="1"
-F 0 "#PWRp0128" H 5150 2850 30  0001 C CNN
+F 0 "#PWRp0132" H 5150 2850 30  0001 C CNN
 F 1 "GND" H 5150 2780 30  0001 C CNN
 F 2 "" H 5150 2850 60  0000 C CNN
